File: K176IE13.sch (EAGLE design)
At the start: 59 parts, among them J1 0R-JUMPB

Commit message: .
Parts:
- removed C206: 470m, rcl:CPOL-EUE3.5-8
- removed C207: 100n, rcl:C-EUC0805
- removed DD5: TD62308AF, TD62308:TD62308AF
- removed L202: (no value), rcl:L-US0204/7
- removed SJ1: (no value), jumper:SJ
- added C10, C8: 33n, rcl:C-EUC0805
- added C11, C12, C304: 100n, rcl:C-EUC0805
- added C13: 100n, rcl:C-EUC1206
- added C303: 150, rcl:C-EUC0805
- added C305: 100m, rcl:CPOL-EUE2.5-5
- added C7: 330n, rcl:C-EUC0805
- added C9: 47m, rcl:CPOL-EUE2.5-5
- added D6, D7, D8, D9: (no value), diode:DIODE-SOD80C
- added DA3: MC34063AD, mc34063-2:MC34063AD
- added DD40: 4011D, 40xx:4011D
- added DD50: К176ЛЕ5, 40xx:4001N
- added JP6, JP7: (no value), Разъёмы штырьковые 2.54мм:PINHD-1X1
- added JP8: (no value), Разъёмы штырьковые 2.54мм:PINHD-1X4
- added JP9: (no value), Разъёмы штырьковые 2.54мм:PINHD-1X7
- added L301: min13mkh, rcl:L-USTFI0305
- added R10, R15, R16: 18k, rcl:R-EU_M0805
- added R11: 6k8, rcl:R-EU_M0805
- added R12: (no value), rcl:R-TRIMM3339P
- added R13, R14: 2M, rcl:R-EU_M0805
- added R301: 0.33r, rcl:R-EU_M1206
- added R303: 91k, rcl:R-EU_M0805
- added R304: 1k, rcl:R-EU_M0805
- added R9: 620k, rcl:R-EU_M0805
- added VD301: SS12, diode:SCHOTTKY-DIODESMD
- DD4: value TD62305FB -> ULN2003AN; device uln-udn:ULN2003AD -> uln-udn:ULN2003AN
- R203: value 1k5 -> 2k7
- R204: value 13k -> 62k
Connections:
- removed net +12V: C206.+, C207.1, L202.2
- removed net N$26: DD4.CD+, SJ1.2
- removed net N$46: C204.1, C205.+, L202.1, R204.2, VD201.C
- removed net S1: DD4.O1
- removed net S2: DD4.O2
- removed net S3: DD4.O3
- removed net S4: DD4.O4
- removed net S5: DD4.O5
- removed net S6: DD4.O6
- removed net S7: DD4.O7
- removed net VCC/2: DD5.VCCA, DD5.VCCB, SJ1.1
- new net +24V: C204.1, C205.+, R204.2, VD201.C
- new net N$47: JP6.1, JP7.1
- new net N$48: C7.1, D6.C, DD50A.I0, DD50A.I1, R9.2
- new net N$49: D8.A, DD40D.I1, DD50B.O
- new net N$50: C8.1, D7.A, DD50A.O
- new net N$51: C8.2, DD40D.I0, R10.1
- new net N$52: D7.C, D8.C, DD50C.I0, DD50D.I0, R14.1
- new net N$53: C9.+, DD40D.O
- new net N$54: C9.-, R11.1
- new net N$55: DD50B.I0, DD50B.I1, R11.2, R12.A
- new net N$56: DD40A.O, DD40C.I1
- new net N$57: DD40A.I1, DD50C.I1, DD50D.O, R13.1
- new net N$58: C10.1, DD50D.I1, R13.2
- new net N$59: D6.A
- new net N$60: DD40B.O, DD40C.I0
- new net N$61: C10.2, DD40B.I1, DD50C.O
- new net N$62: DD40A.I0, R16.1
- new net N$63: R10.2, R16.2
- new net N$64: D9.C
- new net N$65: DD4.O3, JP9.5
- new net N$66: D9.A, DD40B.I0, R15.1
- new net N$67: DD4.O2, JP9.6
- new net N$68: DD4.O1, JP9.7
- new net N$76: DA3.FB, R303.2, R304.1
- new net N$78: DA3.DC, DA3.IS, DA3.SWC, R301.2
- new net N$79: DA3.SWE, L301.1, VD301.C
- new net N$80: C303.1, DA3.TC
- new net V-: C303.2, C304.1, C305.-, DA3.GND, R304.2, VD301.A
- net +5V: now also DA3.VCC, R301.1
- net GND: now also C11.2, C12.2, C13.2, C304.2, C305.+, C7.2, L301.2, R12.E, R12.S, R303.1, R9.1; no longer C206.-, C207.2, DD5.GND@1, DD5.GND@2
- net N$18: now also DD3A.G; no longer DD3A.A
- net N$19: now also DD3A.F; no longer DD3A.B
- net N$20: now also DD3A.E; no longer DD3A.C
- net N$22: now also DD3A.C; no longer DD3A.E
- net N$23: now also DD3A.B; no longer DD3A.F
- net N$24: now also DD3A.A; no longer DD3A.G
- net N$31: now also DD4.O7, JP9.1; no longer DD5.O1A
- net N$32: now also DD4.O6, JP9.2; no longer DD5.O2A
- net N$33: now also DD4.O5, JP9.3; no longer DD5.O1B
- net N$34: now also DD4.O4, JP9.4; no longer DD5.O2B
- net T1: now also DD6.I1, JP8.1; no longer DD5.I1A
- net T2: now also DD6.I2, JP8.2; no longer DD5.I2A
- net T3: now also DD6.I3, JP8.3; no longer DD5.I1B
- net T4: now also DD6.I4, JP8.4; no longer DD5.I2B
- net VCC: now also C11.1, C12.1, C13.1
Other:
- note added: "95khz"
- note added: "d e f a b c g"

Commit message: .
Parts:
- added C14: 10n, rcl:C-EUC0805
- added C15: 510, resistor:C-EUC0805K
- added C19: 10u/100V, rcl:CPOL-EUTT5D9L
- added DA1: MC34063AD, mc34063-2:MC34063AD
- added L2, L3: (no value), rcl:L-USIR-2
- added L4: 15uH, rcl:L-US0204/7
- added L6: 150uH, rcl:L-US0204/7
- added R17: 10k, rcl:R-EU_M0805
- added R18: 100k, rcl:R-EU_R0805
- added R19: 2k7, rcl:R-EU_R0805
- added R1A: (no value), resistor:R-EU_R1206
- added R1B: 0.22, resistor:R-EU_R1206
- added R20, R21: 1k, rcl:R-EU_R0805
- added T3: (no value), transistor:-NPN-TO126
- added T4: (no value), transistor:-PNP-TO126
- added VD1: 1N4148, diode:DIODE-SOD80C
- added VD2: FR207, diode:DIODE-DO41-10
- added VT1: КТ3102, transistor-npn:BC338
- added VT2: КТ3107, transistor-pnp:MPSA64
- added VT3: IRF630, transistor-fet:BUZ22
- C303: value 150 -> 200
- R303: value 91k -> 1k
- R304: value 1k -> 90k
Connections:
- net +5V renamed +3V3
- new net N$46: T3.C, T4.B
- new net N$77: DA1.SWE, R20.1, R21.1, VD1.A, VT1.B, VT2.B
- new net N$81: C14.1, R17.1, T3.B
- new net N$82: C14.2, L2.1, T4.C
- new net N$83: C15.1, DA1.TC
- new net N$85: L3.1
- new net N$86: L3.2
- new net N$87: L4.2, VD2.A, VT3.D
- new net N$88: DA1.IS, L6.1, R1A.2, R1B.2
- new net N$89: DA1.FB, R18.1, R19.2
- new net N$90: C19.+, R18.2, VD2.C
- new net N$92: DA1.SWC, DA1.VCC, R1A.1, R1B.1, VT1.C
- new net N$93: DA1.DC, L4.1, L6.2
- new net N$95: R21.2, VD1.C, VT1.E, VT2.E, VT3.G
- new net VCC/2: R17.2, T4.E
- net GND: now also C15.2, C19.-, DA1.GND, L2.2, R19.1, R20.2, T3.E, VT2.C, VT3.S
Other:
- moved on the sheet: JP1, JP2, JP3, JP4, JP5

Commit message: .
Parts:
- removed C303: 200, rcl:C-EUC0805
- removed C304: 100n, rcl:C-EUC0805
- removed C305: 100m, rcl:CPOL-EUE2.5-5
- removed DA3: MC34063AD, mc34063-2:MC34063AD
- removed L301: min13mkh, rcl:L-USTFI0305
- removed L6: 150uH, rcl:L-US0204/7
- removed R301: 0.33r, rcl:R-EU_M1206
- removed R303: 1k, rcl:R-EU_M0805
- removed R304: 90k, rcl:R-EU_M0805
- removed VD301: SS12, diode:SCHOTTKY-DIODESMD
- added JP10: (no value), Разъёмы штырьковые 2.54мм:PINHD-1X7
- added R22, R23: 330, rcl:R-EU_R0805
- L4: value 15uH -> 150uH
Connections:
- removed net N$76: DA3.FB, R303.2, R304.1
- removed net N$78: DA3.DC, DA3.IS, DA3.SWC, R301.2
- removed net N$79: DA3.SWE, L301.1, VD301.C
- removed net N$80: C303.1, DA3.TC
- removed net N$88: DA1.IS, L6.1, R1A.2, R1B.2
- removed net V-: C303.2, C304.1, C305.-, DA3.GND, R304.2, VD301.A
- net +3V3: no longer DA3.VCC, R301.1
- net GND: now also R23.1; no longer C304.2, C305.+, L301.2, R303.1
- net N$18: now also DD3A.A, JP9.1; no longer DD3A.G, DD4.I1
- net N$19: now also DD3A.B, JP9.2; no longer DD3A.F, DD4.I2
- net N$20: now also DD3A.C, JP9.3; no longer DD3A.E, DD4.I3
- net N$21: now also JP9.4; no longer DD4.I4
- net N$22: now also DD3A.E, JP9.5; no longer DD3A.C, DD4.I5
- net N$23: now also DD3A.F, JP9.6; no longer DD3A.B, DD4.I6
- net N$24: now also DD3A.G, JP9.7; no longer DD3A.A, DD4.I7
- net N$31: now also DD4.I7, JP10.1; no longer DD4.O7, JP9.1
- net N$32: now also DD4.I6, JP10.2; no longer DD4.O6, JP9.2
- net N$33: now also DD4.I5, JP10.3; no longer DD4.O5, JP9.3
- net N$34: now also DD4.I4, JP10.4; no longer DD4.O4, JP9.4
- net N$65: now also DD4.I3, JP10.5; no longer DD4.O3, JP9.5
- net N$67: now also DD4.I2, JP10.6; no longer DD4.O2, JP9.6
- net N$68: now also DD4.I1, JP10.7; no longer DD4.O1, JP9.7
- net N$77: now also R22.1, R22.2, R23.2
- net N$93: now also DA1.IS, R1A.2, R1B.2; no longer L6.2
Other:
- note removed: "95khz"
- moved on the sheet: C15, C19, DA1, DD4, JP1, JP2, JP3, JP4, JP5, JP9, L4, R18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

Commit message: .
Parts:
- removed C15: 510, resistor:C-EUC0805K
- removed C19: 10u/100V, rcl:CPOL-EUTT5D9L
- removed DA1: MC34063AD, mc34063-2:MC34063AD
- removed L4: 150uH, rcl:L-US0204/7
- removed R18: 100k, rcl:R-EU_R0805
- removed R19: 2k7, rcl:R-EU_R0805
- removed R1A: (no value), resistor:R-EU_R1206
- removed R1B: 0.22, resistor:R-EU_R1206
- removed R20, R21: 1k, rcl:R-EU_R0805
- removed R22, R23: 330, rcl:R-EU_R0805
- removed VD1: 1N4148, diode:DIODE-SOD80C
- removed VD2: FR207, diode:DIODE-DO41-10
- removed VT1: КТ3102, transistor-npn:BC338
- removed VT2: КТ3107, transistor-pnp:MPSA64
- removed VT3: IRF630, transistor-fet:BUZ22
- added C17: 10u/100V, rcl:CPOL-EUTT5D9L
- added C18: 510, resistor:C-EUC0805K
- added DA3: MC34063AD, mc34063:MC34063TAD
- added L5: 150uH, rcl:L-US0204/7
- added R1B1, R1B2: 0.22, resistor:R-EU_R1206
- added R24: 15k, rcl:R-EU_R0805
- added R25, R27: 1k, rcl:R-EU_R0805
- added R28: 330, rcl:R-EU_R0805
- added R29: 1k(330), rcl:R-EU_R0805
- added VD3: FR207, diode:DIODE-DO41-10
- added VD4: 1N4148, diode:DIODE-SOD80C
- added VT4: КТ3107, transistor-pnp:MPSA64
- added VT5: IRF630, transistor-fet:BUZ22
- added VT6: КТ3102, transistor-npn:BC338
Connections:
- removed net N$77: DA1.SWE, R20.1, R21.1, R22.1, R22.2, R23.2, VD1.A, VT1.B, VT2.B
- removed net N$83: C15.1, DA1.TC
- removed net N$87: L4.2, VD2.A, VT3.D
- removed net N$89: DA1.FB, R18.1, R19.2
- removed net N$90: C19.+, R18.2, VD2.C
- removed net N$95: R21.2, VD1.C, VT1.E, VT2.E, VT3.G
- new net N$79: DA3.SWE, R27.1, R28.1, R28.2, R29.2, VD4.A, VT4.B, VT6.B
- new net N$88: L5.2, VD3.A, VT5.D
- new net N$91: DA3.FB, R24.1, R25.2
- new net N$94: DA3.IS, L5.1, R1B1.2
- new net N$96: DA3.DC, DA3.SWC, DA3.VCC, R1B1.1, R1B2.1, R1B2.2, VT6.C
- new net N$98: C18.1, DA3.TC
- net GND: now also C17.-, C18.2, DA3.GND, R25.1, R29.1, VT4.C, VT5.S; no longer C15.2, C19.-, DA1.GND, R19.1, R20.2, R23.1, VT2.C, VT3.S
- net N$92: now also C17.+, R24.2, VD3.C; no longer DA1.SWC, DA1.VCC, R1A.1, R1B.1, VT1.C
- net N$93: now also R27.2, VD4.C, VT4.E, VT5.G, VT6.E; no longer DA1.DC, DA1.IS, L4.1, R1A.2, R1B.2
Other:
- moved on the sheet: C14, C201, C202, C203, C204, C205, DA2, JP6, JP7, L2, L201, L3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

Commit message: .
Parts:
- removed VT5: IRF630, transistor-fet:BUZ22
- added VT1: (no value), m_transistor:MOSFET-N_DPACK
- DD4: value ULN2003AN -> TD62305FB; device uln-udn:ULN2003AN -> uln-udn:ULN2003AD
Connections:
- net GND: now also VT1.S; no longer DD4.GND, VT5.S
- net N$31: now also DD4.I1; no longer DD4.I7
- net N$32: now also DD4.I2; no longer DD4.I6
- net N$33: now also DD4.I3; no longer DD4.I5
- net N$65: now also DD4.I5; no longer DD4.I3
- net N$67: now also DD4.I6; no longer DD4.I2
- net N$68: now also DD4.I7; no longer DD4.I1
- net N$88: now also VT1.D; no longer VT5.D
- net N$93: now also VT1.G; no longer VT5.G
Other:
- moved on the sheet: C17, C18, DA3, DD4, JP10, L5, R1B1, R1B2, R24, R25, R27, R28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

Commit message: .
Parts:
- removed JP1, JP2, JP3, JP4, JP5: (no value), Разъёмы штырьковые 2.54мм:PINHD-2X4
- added S4, S6, S7, S8, S9: SKHMPSE010, switch:SKHMPSE010
- added U$8: IV-6_T, vfd:IV-6_T
- added XH, XH1, XH2, XH3, XH4: IV-6, ie13:CON_VFD_IV-6
Other:
- note added: "11 5 4 3 2 1 6 7 8 9 10"
- note added: "20v"

Commit message: .
Parts:
- removed S4, S6: SKHMPSE010, switch:SKHMPSE010
- removed U$8: IV-6_T, vfd:IV-6_T
- removed XH, XH1, XH2, XH3, XH4: IV-6, ie13:CON_VFD_IV-6
- added V1, V2, V3, V4, V5, V6: ИВ-6, vfd:IV-6_T_P
- S1: value M -> SKHMPSE010; device switch-omron:10-XX -> switch:SKHMPSE010
- S2: value Ч -> SKHMPSE010; device switch-omron:10-XX -> switch:SKHMPSE010
Connections:
- new net A: V1.D, V2.D, V4.D, V5.D
- new net B: V1.E, V2.E, V4.E, V5.E
- new net C: V1.F, V2.F, V4.F, V5.F
- new net D: V1.A, V2.A, V4.A, V5.A
- new net E: V1.B, V2.B, V4.B, V5.B
- new net F: V1.C, V2.C, V4.C, V5.C
- new net G: V1.G, V2.G, V4.G, V5.G
- new net H1: V1.H
- new net H2: V2.H
- new net H3: V4.H
- new net H4: V5.H
- new net HE: V1.H1, V2.H1, V4.H1, V5.H1
- new net HK: V1.H2K, V2.H2K, V4.H2K, V5.H2K
- new net S1: V1.S
- new net S2: V2.S
- new net S3: V4.S
- new net S4: V5.S
- net N$12: now also S1.2.1, S1.2.2, S2.2.1, S2.2.2; no longer S1.S, S1.S1, S2.S, S2.S1
- net N$4: now also S2.1.1, S2.1.2; no longer S2.P, S2.P1
- net N$9: now also S1.1.1, S1.1.2; no longer S1.P, S1.P1
Other:
- note removed: "11 5 4 3 2 1 6 7 8 9 10"

Commit message: .
Parts:
- removed S7, S8, S9: SKHMPSE010, switch:SKHMPSE010
- added R18: 10k, rcl:R-EU_M0805
- C203: value 470 -> 120
- L201: value 100mkhn -> 50mkhn
- S1: value SKHMPSE010 -> Ч
- S2: value SKHMPSE010 -> М
- V3: value ИВ-6 -> ИВ-3А
Connections:
- removed net +24V: C204.1, C205.+, R204.2, VD201.C
- removed net N$28: C5.1, JP19.1, L1.2, U$13.EN, U$13.IN
- removed net N$96: DA3.DC, DA3.SWC, DA3.VCC, R1B1.1, R1B2.1, R1B2.2, VT6.C
- new net +30V: C204.1, C205.+, R18.2, R204.2, VD201.C
- new net N$26: DA3.DC, DA3.SWC, R18.1, R1B2.1, R1B2.2, VT6.C
- net +3V3: now also C5.1, DA3.VCC, JP19.1, L1.2, R1B1.1, U$13.EN, U$13.IN
Other:
- note added: "+6v"
- moved on the sheet: C1, C14, C17, C18, C2, C201, C202, C203, C204, C205, C5, C6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
