File: K176IE13.sch (EAGLE design)
At the start: 104 parts, among them J1 0R-JUMPB

Commit message: .
Parts:
- added C15, C16: 22n, rcl:C-EUC1206
- added C19: 120, rcl:C-EUC0805
- added C20, C21, C24: 100n, rcl:C-EUC0805
- added C22: 100m, rcl:CPOL-EUE2.5-5
- added C23: 470m, rcl:CPOL-EUE3.5-8
- added C25, C26: 33, rcl:C-EU025-025X050
- added C27: 2n2, rcl:C-EU025-025X050
- added C28, C29: 100m, rcl:CPOL-EUE2-5
- added C30: 1m, rcl:C-EU025-025X050
- added D10, D11: (no value), diode:DIODE-SOD80C
- added D12: (no value), diode:ZENER-DIODEDO34-7
- added DA1: MC34063AD, mc34063-2:MC34063AD
- added DA4: LM311,К554СА3KY, IC:LM311,К554СА3KY
- added IV1, IV2, IV3, IV6: 24r, rcl:R-EU_M0805
- added IV3A: 17r, rcl:R-EU_M0805
- added L4, L6, L7: (no value), rcl:L-USL3225M
- added L8, L9: 50mkhn, rcl:L-USTFI0305
- added R: (no value), rcl:R-EU_M0805
- added R19, R33: 100k, rcl:R-EU_M0805
- added R20, R21: 56k, rcl:R-EU_M0805
- added R22, R23: 8k2, rcl:R-EU_M0805
- added R26: 180, rcl:R-EU_M0805
- added R30: 0.33r, rcl:R-EU_M1206
- added R31: 470, rcl:R-EU_M0805
- added R32: 1k, rcl:R-EU_M0805
- added R34, R35: 47k, rcl:R-EU_0207/10
- added R36: 1k, rcl:R-EU_0207/10
- added R37: 30k, rcl:R-EU_0207/10
- added R38, R39, R40: 15k, rcl:R-EU_0207/10
- added R41, R42: 220, rcl:R-EU_0207/10
- added R43: 10k, rcl:R-EU_0207/10
- added VT10, VT8: BJT_NPN_TO-92_CBE, m_transistor:BJT_NPN_TO-92_CBE
- added VT11, VT9: BJT_PNP_TO-92_CBE, m_transistor:BJT_PNP_TO-92_CBE
- added VT2, VT7: (no value), m_transistor:MOSFET-N_DPACK
- added VT3, VT5: КТ3102, transistor-npn:BC338
Connections:
- new net -24V: C30.1, D12.A
- new net N$100: IV3A.2, R.1
- new net N$101: C28.+, R37.2, R38.2, VT10.E, VT11.E
- new net N$102: C25.2, C26.1, DA4.OUT, R34.1, R35.2, R36.1
- new net N$103: C25.1, R34.2, VT9.B
- new net N$104: C26.2, R35.1, VT8.B
- new net N$105: C30.2, D12.C, R41.1, R42.2, R43.2
- new net N$106: C28.-, R41.2
- new net N$107: C29.-, R42.1
- new net N$109: DA4.-IN, R37.1, R39.2, R40.1
- new net N$110: C27.1, DA4.+IN, R38.1
- new net N$28: C16.1, L4.2, VT5.C
- new net N$69: R19.1, VT2.G
- new net N$70: C203.2, DA2.GND, DA2.SWE, VT2.D
- new net N$71: C15.2, L6.1, VT3.C
- new net N$72: R20.1, R22.1, VT5.B
- new net N$73: R21.1, R23.1, VT3.B
- new net N$74: DA1.DC, R26.2
- new net N$75: L4.1, L6.2, R22.2, R23.2
- new net N$76: C16.2, R21.2
- new net N$78: DA1.IS, L8.1, R26.1, R30.2
- new net N$80: C15.1, R20.2
- new net N$83: VT10.B, VT11.B, VT8.C, VT9.C
- new net N$87: C19.1, DA1.TC
- new net N$89: C24.1, DA1.FB, R31.1, R32.2
- new net N$90: D10.A, L9.2
- new net N$95: R33.1, VT7.G
- new net N$96: C20.2, C22.-, D11.C, IV1.1, IV2.1, IV3.1, IV3A.1, IV6.1
- new net N$97: D10.C, R31.2
- new net N$99: C20.1, C22.+, DA1.SWC, IV1.2, IV2.2, IV3.2, IV6.2, L8.2, L9.1, R.2
- new net V+: DA4.V+, R36.2, R40.2, VT10.C, VT9.E
- net +3V3: now also C21.1, C23.+, DA1.VCC, R30.1
- net GND: now also C19.2, C21.2, C23.-, C24.2, C27.2, C29.+, D11.A, DA1.GND, DA1.SWE, DA4.GND, DA4.V-, R19.2, R32.1, R33.2, R39.1, R43.1, VT11.C, VT2.S, VT3.E, VT5.E, VT7.S, VT8.E; no longer C203.2, DA2.GND, DA2.SWE
Other:
- note added: "1.25в"
- note added: "1.8в"
- moved on the sheet: C201, C202, C203, C204, C205, DA2, JP6, JP7, L201, R201, R202, R203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

Commit message: .
Parts:
- added C31: 100m, rcl:CPOL-EUE2-5
- added R46: 1k, rcl:R-EU_M0805
- added R47: 270, rcl:R-EU_M0805
- added U$24: TRAN_EE16, ie13:TRAN_EE16
- added VT14, VT15: BC847, m_transistor:BJT_NPN_SOT23_BCE
- R36, R39: device rcl:R-EU_0207/10 -> rcl:R-EU_M0805
Connections:
- new net N$116: U$24.1, VT15.C
- new net N$117: U$24.3, VT14.C
- new net N$118: U$24.2, VT14.B
- new net N$119: U$24.6, VT15.B
- new net N$120: R46.1, U$24.5
- new net N$121: C31.-, R46.2, R47.2, U$24.4
- net GND: now also C31.+, R47.1, VT14.E, VT15.E

Commit message: .
Parts:
- added R44: 0, rcl:R-EU_R1206
- added U$7: TRAN_EE16, ie13:TRAN_EE16
- C31: device rcl:CPOL-EUE2-5 -> rcl:CPOL-EUSANYO_SMD_A5
Connections:
- removed net +3V3: C201.+, C202.1, C21.1, C23.+, C5.1, DA1.VCC, DA2.VCC, DA3.VCC, JP19.1, L1.2, R1B1.1, R201.1, R30.1, U$13.EN, U$13.IN
- removed net N$120: R46.1, U$24.5
- new net +3V7: C201.+, C202.1, C21.1, C23.+, C5.1, DA1.VCC, DA2.VCC, DA3.VCC, JP19.1, L1.2, R1B1.1, R201.1, R30.1, R46.1, U$13.EN, U$13.IN, U$24.3
- new net HE3: V3.H1
- new net HK3: V3.H2K
- new net N$77: R44.1, VT14.E
- net GND: now also R44.2; no longer VT14.E
- net N$117: now also U$24.2; no longer U$24.3
- net N$118: now also U$24.5; no longer U$24.2
Other:
- moved on the sheet: C14, C15, C16, C31, C5, C6, D5, DD4, JP10, JP19, L1, L2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

Commit message: >d
Parts:
- removed C15, C16: 22n, rcl:C-EUC1206
- removed C17: 10u/100V, rcl:CPOL-EUTT5D9L
- removed C18: 510, resistor:C-EUC0805K
- removed C19: 120, rcl:C-EUC0805
- removed C20, C21, C24: 100n, rcl:C-EUC0805
- removed C22: 100m, rcl:CPOL-EUE2.5-5
- removed C23: 470m, rcl:CPOL-EUE3.5-8
- removed C25, C26: 33, rcl:C-EU025-025X050
- removed C27: 2n2, rcl:C-EU025-025X050
- removed C28, C29: 100m, rcl:CPOL-EUE2-5
- removed C30: 1m, rcl:C-EU025-025X050
- removed C31: 100m, rcl:CPOL-EUSANYO_SMD_A5
- removed D10, D11: (no value), diode:DIODE-SOD80C
- removed D12: (no value), diode:ZENER-DIODEDO34-7
- removed DA1: MC34063AD, mc34063-2:MC34063AD
- removed DA3: MC34063AD, mc34063:MC34063TAD
- removed DA4: LM311,К554СА3KY, IC:LM311,К554СА3KY
- removed IV1, IV2, IV3, IV6: 24r, rcl:R-EU_M0805
- removed IV3A: 17r, rcl:R-EU_M0805
- removed JP10: (no value), Разъёмы штырьковые 2.54мм:PINHD-1X7
- removed L2, L3: (no value), rcl:L-USIR-2
- removed L4, L6, L7: (no value), rcl:L-USL3225M
- removed L5: 150uH, rcl:L-US0204/7
- removed L8, L9: 50mkhn, rcl:L-USTFI0305
- removed R: (no value), rcl:R-EU_M0805
- removed R1B1, R1B2: 0.22, resistor:R-EU_R1206
- removed R22, R23: 8k2, rcl:R-EU_M0805
- removed R24: 15k, rcl:R-EU_R0805
- removed R25, R27: 1k, rcl:R-EU_R0805
- removed R26: 180, rcl:R-EU_M0805
- removed R28: 330, rcl:R-EU_R0805
- removed R29: 1k(330), rcl:R-EU_R0805
- removed R30: 0.33r, rcl:R-EU_M1206
- removed R31: 470, rcl:R-EU_M0805
- removed R32, R36, R46: 1k, rcl:R-EU_M0805
- removed R33: 100k, rcl:R-EU_M0805
- removed R34, R35: 47k, rcl:R-EU_0207/10
- removed R37: 30k, rcl:R-EU_0207/10
- removed R38, R40: 15k, rcl:R-EU_0207/10
- removed R39: 15k, rcl:R-EU_M0805
- removed R41, R42: 220, rcl:R-EU_0207/10
- removed R43: 10k, rcl:R-EU_0207/10
- removed R44: 0, rcl:R-EU_R1206
- removed R47: 270, rcl:R-EU_M0805
- removed T3: (no value), transistor:-NPN-TO126
- removed T4: (no value), transistor:-PNP-TO126
- removed U$24: TRAN_EE16, ie13:TRAN_EE16
- removed V6: ИВ-6, vfd:IV-6_T_P
- removed VD3: FR207, diode:DIODE-DO41-10
- removed VD4: 1N4148, diode:DIODE-SOD80C
- removed VT10, VT8: BJT_NPN_TO-92_CBE, m_transistor:BJT_NPN_TO-92_CBE
- removed VT11, VT9: BJT_PNP_TO-92_CBE, m_transistor:BJT_PNP_TO-92_CBE
- removed VT14, VT15: BC847, m_transistor:BJT_NPN_SOT23_BCE
- removed VT4: КТ3107, transistor-pnp:MPSA64
- removed VT5, VT6: КТ3102, transistor-npn:BC338
- removed VT7: (no value), m_transistor:MOSFET-N_DPACK
- added JP1: (no value), Разъёмы штырьковые 2.54мм:PINHD-1X7
- added T19: (no value), transistor:-NPN-TO92-ECB
- added U$9: MOD_TP4056, TP4056+mod:MOD_TP4056
- C14: value 10n -> (none); device rcl:C-EUC0805 -> rcl:C-EUC1206
- C5: value (none) -> 10m; device rcl:C-EUC1206 -> rcl:CPOL-EUSANYO_SMD_A5
- R17: value 10k -> (none); device rcl:R-EU_M0805 -> rcl:R-TRIMM3296W
- R18: value 10k -> 68k
- R20: value 56k -> 2k2
- R21: value 56k -> (none)
- R6: value (none) -> 1k; device rcl:R-TRIMM3296W -> rcl:R-EU_M0805
- R7: value 68k -> 270
- R8: value 2k2 -> 0; device rcl:R-EU_M0805 -> rcl:R-EU_M1206
- T1: value (none) -> TRAN_EE16; device transistor:-NPN-TO92-ECB -> ie13:TRAN_EE16
- VT1: value (none) -> BC847; device m_transistor:MOSFET-N_DPACK -> m_transistor:BJT_NPN_SOT23_BCE
- VT3: value КТ3102 -> BC847; device transistor-npn:BC338 -> m_transistor:BJT_NPN_SOT23_BCE
Connections:
- removed net -24V: C30.1, D12.A
- removed net N$100: IV3A.2, R.1
- removed net N$101: C28.+, R37.2, R38.2, VT10.E, VT11.E
- removed net N$102: C25.2, C26.1, DA4.OUT, R34.1, R35.2, R36.1
- removed net N$103: C25.1, R34.2, VT9.B
- removed net N$104: C26.2, R35.1, VT8.B
- removed net N$105: C30.2, D12.C, R41.1, R42.2, R43.2
- removed net N$106: C28.-, R41.2
- removed net N$107: C29.-, R42.1
- removed net N$109: DA4.-IN, R37.1, R39.2, R40.1
- removed net N$110: C27.1, DA4.+IN, R38.1
- removed net N$34 (its old number): DD4.I4, JP10.4
- removed net N$46: T3.C, T4.B
- removed net N$71: C15.2, L6.1, VT3.C
- removed net N$72: R20.1, R22.1, VT5.B
- removed net N$73: R21.1, R23.1, VT3.B
- removed net N$74: DA1.DC, R26.2
- removed net N$75: L4.1, L6.2, R22.2, R23.2
- removed net N$76: C16.2, R21.2
- removed net N$77: R44.1, VT14.E
- removed net N$78: DA1.IS, L8.1, R26.1, R30.2
- removed net N$79: DA3.SWE, R27.1, R28.1, R28.2, R29.2, VD4.A, VT4.B, VT6.B
- removed net N$80: C15.1, R20.2
- removed net N$81: C14.1, R17.1, T3.B
- removed net N$82: C14.2, L2.1, T4.C
- removed net N$83: VT10.B, VT11.B, VT8.C, VT9.C
- removed net N$85: L3.1
- removed net N$86: L3.2
- removed net N$87: C19.1, DA1.TC
- removed net N$88: L5.2, VD3.A, VT1.D
- removed net N$89: C24.1, DA1.FB, R31.1, R32.2
- removed net N$90: D10.A, L9.2
- removed net N$91: DA3.FB, R24.1, R25.2
- removed net N$92: C17.+, R24.2, VD3.C
- removed net N$93: R27.2, VD4.C, VT1.G, VT4.E, VT6.E
- removed net N$94: DA3.IS, L5.1, R1B1.2
- removed net N$95: R33.1, VT7.G
- removed net N$96: C20.2, C22.-, D11.C, IV1.1, IV2.1, IV3.1, IV3A.1, IV6.1
- removed net N$97: D10.C, R31.2
- removed net N$98: C18.1, DA3.TC
- removed net N$99: C20.1, C22.+, DA1.SWC, IV1.2, IV2.2, IV3.2, IV6.2, L8.2, L9.1, R.2
- removed net V+: DA4.V+, R36.2, R40.2, VT10.C, VT9.E
- removed net VCC/2: R17.2, T4.E
- new net +3V3: C6.1, JP19.1, L1.2, U$13.EN, U$13.IN
- new net N$27: C5.+, R7.1, R8.2, VT1.E, VT3.E
- new net SD: R21.2, V3.S
- net +30V: now also R21.1; no longer R18.2
- net +3V7: now also R6.1, T1.5; no longer C21.1, C23.+, C5.1, DA1.VCC, DA3.VCC, JP19.1, L1.2, R1B1.1, R30.1, R46.1, U$13.EN, U$13.IN, U$24.3
- net GND: now also C14.2, R20.1; no longer C17.-, C18.2, C19.2, C21.2, C23.-, C24.2, C27.2, C29.+, C31.+, C5.2, D11.A, DA1.GND, DA1.SWE, DA3.GND, DA4.GND, DA4.V-, L2.2, R25.1, R29.1, R32.1, R33.2, R39.1, R43.1, R44.2, R47.1, R8.1, T3.E, VT1.S, VT11.C, VT15.E, VT3.E, VT4.C, VT5.E, VT7.S, VT8.E
- net N$116: now also T1.1, VT1.C; no longer U$24.1, VT15.C
- net N$117: now also T1.3, VT3.C; no longer U$24.2, VT14.C
- net N$118: now also T1.2, VT3.B; no longer U$24.5, VT14.B
- net N$119: now also T1.6, VT1.B; no longer U$24.6, VT15.B
- net N$121: now also C5.-, R6.2, R7.2, T1.4; no longer C31.-, R46.2, R47.2, U$24.4
- net N$17: now also T19.E; no longer T1.E
- net N$26: now also DD4.I4, JP1.4; no longer DA3.DC, DA3.SWC, R18.1, R1B2.1, R1B2.2, VT6.C
- net N$28: now also R8.1, VT2.D; no longer C16.1, L4.2, VT5.C
- net N$31: now also JP1.1; no longer JP10.1
- net N$32: now also JP1.2; no longer JP10.2
- net N$33: now also JP1.3; no longer JP10.3
- net N$36: now also T19.B; no longer T1.B
- net N$43: now also R17.E, R18.1; no longer R6.E, R7.1
- net N$44: now also R17.S; no longer R6.S
- net N$45: now also R17.A, R20.2; no longer R6.A, R8.2
- net N$65: now also JP1.5; no longer JP10.5
- net N$67: now also JP1.6; no longer JP10.6
- net N$68: now also JP1.7; no longer JP10.7
- net N$70: no longer VT2.D
- net VCC: now also C14.1, R18.2, T19.C; no longer C6.1, R7.2, T1.C
Other:
- note added: "T1"
- note removed: "+6v"
- note removed: "1.25в"
- note removed: "1.8в"
- note removed: "20v"
- moved on the sheet: C14, C6, D5, JP19, L1, R18, R19, R20, R7, R8, U$13, VT2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

Commit message: .
Parts:
- S3, S4.1, S5: device switch-omron:10-XX -> switch:SKHMPSE010
Connections:
- net N$11: now also S5.1.1, S5.1.2; no longer S5.P, S5.P1
- net N$12: now also S3.1.1, S3.1.2; no longer S3.P, S3.P1
- net N$13: now also S4.1.1.1, S4.1.1.2; no longer S4.1.P, S4.1.P1
- net N$15: now also S3.2.1, S3.2.2, S4.1.2.1, S4.1.2.2; no longer S3.S, S3.S1, S4.1.S, S4.1.S1
- net VCC: now also S5.2.1, S5.2.2; no longer S5.S, S5.S1
Other:
- moved on the sheet: C3, D2, D3, D4, R3, S2

Commit message: b
Parts:
- removed V3: ИВ-3А, vfd:IV-6_T_P
- added U$4: IV-3T_VIXC, vfd:IV-3T_VIXC
- V1, V5: device vfd:IV-6_T_P -> vfd:IV-6_T_VIXC
- V2: value ИВ-6 -> IV-6_T_VIXL; device vfd:IV-6_T_P -> vfd:IV-6_T_VIXL
Connections:
- net HE3: now also U$4.H1; no longer V3.H1
- net HK3: now also U$4.H2K; no longer V3.H2K
- net SD: now also U$4.S; no longer V3.S

Commit message: .
Parts:
- V2: value IV-6_T_VIXL -> ИВ-6
- V3: value IV-3T_VIXC -> ИВ-3А
- V4: device vfd:IV-6_T_P -> vfd:IV-6_T_VIXR
- renumbered U$4 to V3

Commit message: .
Parts:
- removed JP19: (no value), Разъёмы штырьковые 2.54мм:PINHD-1X2/2
- removed JP6, JP7: (no value), Разъёмы штырьковые 2.54мм:PINHD-1X1
- removed U$7: TRAN_EE16, ie13:TRAN_EE16
- added JP2: (no value), Разъёмы штырьковые 2.54мм:PINHD-1X4
- added R22, R23: (no value), rcl:R-EU_M0805
- added T3: TRAN_EE16, ie13:TRAN_EE16
- added XBAT: (no value), Разъёмы штырьковые 2.54мм:PINHD-1X2/2
- DD1: device К176:К176ИЕ12,ИЕ18 -> К176:К176ИЕ12
Connections:
- new net N$46: U$9.P2+B, XBAT.1
- new net N$71: R23.1
- new net N$72: DD6.I4, JP2.1
- new net N$73: DD6.I5, JP2.2
- new net N$74: DD6.I6, JP2.3
- new net N$75: DD6.I7, JP2.4
- net +3V3: now also U$9.P2+OUT; no longer JP19.1
- net GND: now also C203.2, DA2.GND, DA2.SWE, U$9.P2-OUT; no longer JP19.2
- net HE3: now also R22.2
- net HK3: now also R23.2
- net N$47: now also U$9.P2-B, XBAT.2; no longer JP6.1, JP7.1
- net N$70: now also R22.1; no longer C203.2, DA2.GND, DA2.SWE
- net T1: no longer DD6.I1
- net T2: now also JP8.4; no longer DD6.I2, JP8.2
- net T3: now also JP8.2; no longer DD6.I3, JP8.3
- net T4: now also JP8.3; no longer DD6.I4, JP8.4
Other:
- moved on the sheet: C10, C14, C5, C6, D5, DD4, DD40A, DD40B, DD40C, DD50C, DD50D, DD6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
