File: K176IE13.sch (EAGLE design)
At the start: 93 parts, among them J1 0R-JUMPB, T1 TRAN_EE16, T3 TRAN_EE16

Commit message: .
Parts:
- removed T3: TRAN_EE16, ie13:TRAN_EE16
Changed lines of the file:
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@@
 <grid distance="0.1" unitdist="inch" unit="inch" style="lines" multiple="1" display="yes" altdistance="0.01" altunitdist="inch" altunit="inch"/>
 <layers>
-<layer number="1" name="Top" color="4" fill="1" visible="yes" active="no"/>
-<layer number="2" name="Route2" color="1" fill="3" visible="yes" active="no"/>
-<layer number="3" name="Route3" color="4" fill="3" visible="yes" active="no"/>
-<layer number="4" name="Route4" color="1" fill="4" visible="yes" active="no"/>
-<layer number="5" name="Route5" color="4" fill="4" visible="yes" active="no"/>
-<layer number="6" name="Route6" color="1" fill="8" visible="yes" active="no"/>
-<layer number="7" name="Route7" color="4" fill="8" visible="yes" active="no"/>
-<layer number="8" name="Route8" color="1" fill="2" visible="yes" active="no"/>
-<layer number="9" name="Route9" color="4" fill="2" visible="yes" active="no"/>
-<layer number="10" name="Route10" color="1" fill="7" visible="yes" active="no"/>
-<layer number="11" name="Route11" color="4" fill="7" visible="yes" active="no"/>
-<layer number="12" name="Route12" color="1" fill="5" visible="yes" active="no"/>
-<layer number="13" name="Route13" color="4" fill="5" visible="yes" active="no"/>
-<layer number="14" name="Route14" color="1" fill="6" visible="yes" active="no"/>
-<layer number="15" name="Route15" color="4" fill="6" visible="yes" active="no"/>
-<layer number="16" name="Bottom" color="1" fill="1" visible="yes" active="no"/>
-<layer number="17" name="Pads" color="2" fill="1" visible="yes" active="no"/>
-<layer number="18" name="Vias" color="2" fill="1" visible="yes" active="no"/>
-<layer number="19" name="Unrouted" color="6" fill="1" visible="yes" active="no"/>
-<layer number="20" name="Dimension" color="15" fill="1" visible="yes" active="no"/>
-<layer number="21" name="tPlace" color="7" fill="1" visible="yes" active="no"/>
-<layer number="22" name="bPlace" color="7" fill="1" visible="yes" active="no"/>
-<layer number="23" name="tOrigins" color="15" fill="1" visible="yes" active="no"/>
-<layer number="24" name="bOrigins" color="15" fill="1" visible="yes" active="no"/>
-<layer number="25" name="tNames" color="7" fill="1" visible="yes" active="no"/>
-<layer number="26" name="bNames" color="7" fill="1" visible="yes" active="no"/>
-<layer number="27" name="tValues" color="7" fill="1" visible="yes" active="no"/>
-<layer number="28" name="bValues" color="7" fill="1" visible="yes" active="no"/>
+<layer number="1" name="Top" color="4" fill="1" visible="no" active="no"/>
+<layer number="2" name="Route2" color="1" fill="3" visible="no" active="no"/>
+<layer number="3" name="Route3" color="4" fill="3" visible="no" active="no"/>
+<layer number="4" name="Route4" color="1" fill="4" visible="no" active="no"/>
+<layer number="5" name="Route5" color="4" fill="4" visible="no" active="no"/>
+<layer number="6" name="Route6" color="1" fill="8" visible="no" active="no"/>
+<layer number="7" name="Route7" color="4" fill="8" visible="no" active="no"/>
+<layer number="8" name="Route8" color="1" fill="2" visible="no" active="no"/>
+<layer number="9" name="Route9" color="4" fill="2" visible="no" active="no"/>
+<layer number="10" name="Route10" color="1" fill="7" visible="no" active="no"/>
+<layer number="11" name="Route11" color="4" fill="7" visible="no" active="no"/>
+<layer number="12" name="Route12" color="1" fill="5" visible="no" active="no"/>
+<layer number="13" name="Route13" color="4" fill="5" visible="no" active="no"/>
+<layer number="14" name="Route14" color="1" fill="6" visible="no" active="no"/>
+<layer number="15" name="Route15" color="4" fill="6" visible="no" active="no"/>
+<layer number="16" name="Bottom" color="1" fill="1" visible="no" active="no"/>
+<layer number="17" name="Pads" color="2" fill="1" visible="no" active="no"/>
+<layer number="18" name="Vias" color="2" fill="1" visible="no" active="no"/>
+<layer number="19" name="Unrouted" color="6" fill="1" visible="no" active="no"/>
+<layer number="20" name="Dimension" color="15" fill="1" visible="no" active="no"/>
+<layer number="21" name="tPlace" color="7" fill="1" visible="no" active="no"/>
+<layer number="22" name="bPlace" color="7" fill="1" visible="no" active="no"/>
+<layer number="23" name="tOrigins" color="15" fill="1" visible="no" active="no"/>
+<layer number="24" name="bOrigins" color="15" fill="1" visible="no" active="no"/>
+<layer number="25" name="tNames" color="7" fill="1" visible="no" active="no"/>
+<layer number="26" name="bNames" color="7" fill="1" visible="no" active="no"/>
+<layer number="27" name="tValues" color="7" fill="1" visible="no" active="no"/>
+<layer number="28" name="bValues" color="7" fill="1" visible="no" active="no"/>
 <layer number="29" name="tStop" color="7" fill="3" visible="no" active="no"/>
 <layer number="30" name="bStop" color="7" fill="6" visible="no" active="no"/>
@@
 <layer number="35" name="tGlue" color="7" fill="4" visible="no" active="no"/>
 <layer number="36" name="bGlue" color="7" fill="5" visible="no" active="no"/>
-<layer number="37" name="tTest" color="7" fill="1" visible="yes" active="no"/>
-<layer number="38" name="bTest" color="7" fill="1" visible="yes" active="no"/>
+<layer number="37" name="tTest" color="7" fill="1" visible="no" active="no"/>
+<layer number="38" name="bTest" color="7" fill="1" visible="no" active="no"/>
 <layer number="39" name="tKeepout" color="4" fill="11" visible="no" active="no"/>
 <layer number="40" name="bKeepout" color="1" fill="11" visible="no" active="no"/>
@@
 <layer number="44" name="Drills" color="7" fill="1" visible="no" active="no"/>
 <layer number="45" name="Holes" color="7" fill="1" visible="no" active="no"/>
-<layer number="46" name="Milling" color="3" fill="1" visible="yes" active="no"/>
-<layer number="47" name="Measures" color="5" fill="1" visible="yes" active="no"/>
-<layer number="48" name="Document" color="7" fill="1" visible="yes" active="no"/>
-<layer number="49" name="Reference" color="7" fill="1" visible="yes" active="no"/>
-<layer number="50" name="dxf" color="7" fill="1" visible="yes" active="no"/>
-<layer number="51" name="tDocu" color="7" fill="1" visible="yes" active="no"/>
-<layer number="52" name="bDocu" color="7" fill="1" visible="yes" active="no"/>
-<layer number="53" name="tGND_GNDA" color="7" fill="9" visible="yes" active="no"/>
-<layer number="54" name="bGND_GNDA" color="1" fill="9" visible="yes" active="no"/>
-<layer number="56" name="wert" color="7" fill="1" visible="yes" active="no"/>
-<layer number="57" name="tCAD" color="7" fill="1" visible="yes" active="no"/>
+<layer number="46" name="Milling" color="3" fill="1" visible="no" active="no"/>
+<layer number="47" name="Measures" color="5" fill="1" visible="no" active="no"/>
+<layer number="48" name="Document" color="7" fill="1" visible="no" active="no"/>
+<layer number="49" name="Reference" color="7" fill="1" visible="no" active="no"/>
+<layer number="50" name="dxf" color="7" fill="1" visible="no" active="no"/>
+<layer number="51" name="tDocu" color="7" fill="1" visible="no" active="no"/>
+<layer number="52" name="bDocu" color="7" fill="1" visible="no" active="no"/>
+<layer number="53" name="tGND_GNDA" color="7" fill="9" visible="no" active="no"/>
+<layer number="54" name="bGND_GNDA" color="1" fill="9" visible="no" active="no"/>
+<layer number="56" name="wert" color="7" fill="1" visible="no" active="no"/>
+<layer number="57" name="tCAD" color="7" fill="1" visible="no" active="no"/>
 <layer number="88" name="SimResults" color="9" fill="1" visible="yes" active="yes"/>
 <layer number="89" name="SimProbes" color="9" fill="1" visible="yes" active="yes"/>
@@
 <part name="U$1" library="supply1v" deviceset="+3V7" device=""/>
 <part name="GND13" library="supply1v" deviceset="GND" device=""/>
-<part name="T3" library="ie13" deviceset="TRAN_EE16" device=""/>
 <part name="R22" library="rcl" deviceset="R-EU_" device="M0805"/>
 <part name="R23" library="rcl" deviceset="R-EU_" device="M0805"/>
@@
 <instance part="FRAME5" gate="G$2" x="175.26" y="-403.86"/>
 <instance part="R6" gate="G$1" x="45.72" y="-337.82" smashed="yes" rot="MR270">
-<attribute name="NAME" x="49.53" y="-334.2386" size="1.778" layer="95" rot="MR180"/>
-<attribute name="VALUE" x="49.53" y="-337.058" size="1.778" layer="96" rot="MR180"/>
-</instance>
-<instance part="VT1" gate="G$1" x="33.02" y="-337.82"/>
-<instance part="VT3" gate="G$1" x="58.42" y="-337.82" rot="MR0"/>
+<attribute name="NAME" x="46.99" y="-336.7786" size="1.778" layer="95" rot="MR180"/>
+<attribute name="VALUE" x="46.99" y="-339.598" size="1.778" layer="96" rot="MR180"/>
+</instance>
+<instance part="VT1" gate="G$1" x="33.02" y="-337.82" smashed="yes">
+<attribute name="NAME" x="25.4" y="-340.36" size="1.778" layer="95"/>
+<attribute name="VALUE" x="25.4" y="-342.9" size="1.778" layer="96"/>
+</instance>
+<instance part="VT3" gate="G$1" x="58.42" y="-337.82" smashed="yes" rot="MR0">
+<attribute name="NAME" x="66.04" y="-340.36" size="1.778" layer="95" rot="MR0"/>
+<attribute name="VALUE" x="66.04" y="-342.9" size="1.778" layer="96" rot="MR0"/>
+</instance>
 <instance part="R7" gate="G$1" x="45.72" y="-353.06" smashed="yes" rot="R90">
 <attribute name="NAME" x="41.91" y="-349.4786" size="1.778" layer="95" rot="R180"/>
@@
 <instance part="U$1" gate="G$1" x="45.72" y="-220.98"/>
 <instance part="GND13" gate="1" x="45.72" y="-241.3" rot="MR0"/>
-<instance part="T3" gate="G$1" x="129.54" y="-363.22"/>
 <instance part="JP2" gate="A" x="88.9" y="60.96" rot="MR0"/>
 </instances>

Commit message: .
Parts:
- C5: value 10m -> (none)
Changed lines of the file:
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@@
 <part name="VT3" library="m_transistor" deviceset="BJT_NPN" device="_SOT23_BCE" value="BC847"/>
 <part name="R7" library="rcl" deviceset="R-EU_" device="M0805" value="270"/>
-<part name="C5" library="rcl" deviceset="CPOL-EU" device="SANYO_SMD_A5" value="10m"/>
+<part name="C5" library="rcl" deviceset="CPOL-EU" device="SANYO_SMD_A5"/>
 <part name="JP1" library="Разъёмы штырьковые 2.54мм" deviceset="PINHD-1X7" device=""/>
 <part name="R8" library="rcl" deviceset="R-EU_" device="M1206" value="0"/>

Commit message: .
Parts:
- added U$2: ULN2003C, DSS:ULN2003C
- added VT4: (no value), m_transistor:MOSFET-P_SOT23
Connections:
- removed net N$27: C5.+, R7.1, R8.2, VT1.E, VT3.E
- removed net N$70: R22.1
- removed net N$71: R23.1
- net +3V3: now also VT4.S
- net +3V7: now also VT4.D
- net GND: now also C5.+, R7.1, VT1.E, VT3.E
- net HE: now also R22.1
- net HK: now also R23.1
Other:
- note added: "T1 EE16 I 1+1 0.5 II 5 III 2 IV"
- note removed: "T1"
- moved on the sheet: R19, R23, R8, VT2

Commit message: .
Parts:
- added JP3, JP4: (no value), Разъёмы штырьковые 2.54мм:PINHD-1X1
Connections:
- new net N$27: C5.+, R7.1, R8.2, VT1.E, VT3.E
- net A: now also DD4.O1
- net B: now also DD4.O2
- net C: now also DD4.O3
- net D: now also DD4.O4
- net E: now also DD4.O5
- net F: now also DD4.O6
- net G: now also DD4.O7
- net GND: now also DD4.GND, R8.1; no longer C5.+, R7.1, VT1.E, VT3.E
- net N$28: now also DD4.CD+; no longer R8.1, VT2.D

Commit message: .
Parts:
- removed JP3, JP4: (no value), Разъёмы штырьковые 2.54мм:PINHD-1X1
- removed R19: 100k, rcl:R-EU_M0805
- removed VT2: (no value), m_transistor:MOSFET-N_DPACK
- added D10, D11: 1N4148DO35-7, diode:1N4148DO35-7
- renumbered JP1 to X2B, JP9 to X2A
Connections:
- new net HVCC: DD4.CD+, R6.1, T1.5, VT4.D
- new net N$70: D10.C, D11.C
- net +3V7: no longer R6.1, T1.5, VT4.D
- net GND: no longer R19.2, VT2.S
- net N$28: now also D11.A; no longer DD4.CD+
- net N$69: now also D10.A; no longer R19.1, VT2.G
Other:
- note added: "HE"
- note added: "HK"

Commit message: .
Parts:
- added U$12, U$14, U$15, U$17, U$19, U$20, U$22, U$23, U$24, U$25, U$26, U$27, U$28, U$29, U$30, U$31, U$32, U$33, U$34, U$4, U$7: PAD, ie13:PAD
- added U$3, U$35: +, ie13:+
Connections:
- net H4 renamed H5
- new net A3: U$20.P$1, U$3.P$1, V3.D
- new net A5: U$28.P$1, V5.D
- new net B3: U$22.P$1, U$3.P$2, U$35.P$1, V3.E
- new net B5: U$29.P$1, V5.E
- new net C3: U$23.P$1, V3.F
- new net C5: U$30.P$1, V5.F
- new net D3: U$24.P$1, V3.A
- new net D5: U$31.P$1, V5.A
- new net E3: U$25.P$1, V3.B
- new net E5: U$32.P$1, V5.B
- new net F3: U$26.P$1, V3.C
- new net F5: U$33.P$1, V5.C
- new net G3: U$27.P$1, U$35.P$2, V3.G
- new net G5: U$34.P$1, V5.G
- net A: now also U$4.P$1; no longer V5.D
- net B: now also U$7.P$1; no longer V5.E
- net C: now also U$12.P$1; no longer V5.F
- net D: now also U$14.P$1; no longer V5.A
- net E: now also U$15.P$1; no longer V5.B
- net F: now also U$17.P$1; no longer V5.C
- net G: now also U$19.P$1; no longer V5.G
- net H3: now also V3.H

Commit message: .
Parts:
- removed JP2: (no value), Разъёмы штырьковые 2.54мм:PINHD-1X4
- added U$36, U$37, U$38, U$39, U$40, U$41, U$42, U$43, U$44, U$45, U$46, U$47, U$48, U$49: PAD, ie13:PAD
- added X1B: (no value), Разъёмы штырьковые 2.54мм:PINHD-1X4
- renumbered JP8 to X1A
Connections:
- removed net A: DD4.O1, U$4.P$1, V1.D, V2.D, V4.D
- removed net B: DD4.O2, U$7.P$1, V1.E, V2.E, V4.E
- removed net C: DD4.O3, U$12.P$1, V1.F, V2.F, V4.F
- removed net D: DD4.O4, U$14.P$1, V1.A, V2.A, V4.A
- removed net E: DD4.O5, U$15.P$1, V1.B, V2.B, V4.B
- removed net F: DD4.O6, U$17.P$1, V1.C, V2.C, V4.C
- removed net G: DD4.O7, U$19.P$1, V1.G, V2.G, V4.G
- new net A1: U$4.P$1, V1.D
- new net A2: U$36.P$1, V2.D
- new net A4: DD4.O1, U$43.P$1, V4.D
- new net B1: U$7.P$1, V1.E
- new net B2: U$37.P$1, V2.E
- new net B4: DD4.O2, U$44.P$1, V4.E
- new net C1: U$12.P$1, V1.F
- new net C2: U$38.P$1, V2.F
- new net C4: DD4.O3, U$45.P$1, V4.F
- new net D1: U$14.P$1, V1.A
- new net D2: U$39.P$1, V2.A
- new net D4: DD4.O4, U$46.P$1, V4.A
- new net E1: U$15.P$1, V1.B
- new net E2: U$40.P$1, V2.B
- new net E4: DD4.O5, U$47.P$1, V4.B
- new net F1: U$17.P$1, V1.C
- new net F2: U$41.P$1, V2.C
- new net F4: DD4.O6, U$48.P$1, V4.C
- new net G1: U$19.P$1, V1.G
- new net G2: U$42.P$1, V2.G
- new net G4: DD4.O7, U$49.P$1, V4.G
- new net H4: V4.H
- net B3: now also DD6.O2
- net D3: now also DD6.O1
- net GND: now also DD6.GND
- net H3: no longer V4.H
- net N$72: now also X1B.1; no longer JP2.1
- net N$73: now also X1B.2; no longer JP2.2
- net N$74: now also X1B.3; no longer JP2.3
- net N$75: now also X1B.4; no longer JP2.4

Commit message: .
Parts:
- added U$50: +, ie13:+
- added U$51, U$52, U$53, U$54, U$55: PAD, ie13:PAD
Connections:
- net N$72 renamed T1B
- net N$73 renamed T3B
- net N$74 renamed T4B
- net N$75 renamed T2B
- new net HE1: U$51.P$1, V1.H1
- new net HE2: U$53.P$1, V2.H1
- new net HK1: U$52.P$1, V1.H2K
- new net HK2: U$54.P$1, V2.H2K
- net A3: now also DD6.O2, U$55.P$1; no longer U$3.P$1
- net B3: no longer DD6.O2, U$3.P$2, U$35.P$1
- net C3: now also U$35.P$1
- net D3: now also U$3.P$1, U$50.P$2
- net E3: now also U$3.P$2
- net G2: now also DD4.O7
- net G3: now also U$50.P$1
- net G4: no longer DD4.O7
- net HE: no longer V1.H1, V2.H1
- net HK: no longer V1.H2K, V2.H2K
Other:
- moved on the sheet: C5, D10, D11, R6, R7, R8, T1, VT1, VT3, VT4
