File: K176IE13.brd (EAGLE design)
At the start: 113 parts

Commit message: .
Parts:
- added C15, C16: 22n, rcl:C1206
- added C19: 120, rcl:C0805
- added C20, C21, C24: 100n, rcl:C0805
- added C22: 100m, rcl:E2,5-5
- added C23: 470m, rcl:E3,5-8
- added C25, C26: 33, rcl:C025-025X050
- added C27: 2n2, rcl:C025-025X050
- added C28, C29: 100m, rcl:E2-5
- added C30: 1m, rcl:C025-025X050
- added D10, D11: (no value), diode:SOD80C
- added D12: (no value), diode:DO34Z7
- added DA1: MC34063AD, mc34063-2:SOIC8
- added DA4: LM311,К554СА3KY, IC:DIL14
- added IV1, IV2, IV3, IV6: 24r, rcl:M0805
- added IV3A: 17r, rcl:M0805
- added L4, L6, L7: (no value), rcl:L3225M
- added L8, L9: 50mkhn, rcl:TFI0305
- added R: (no value), rcl:M0805
- added R19, R33: 100k, rcl:M0805
- added R20, R21: 56k, rcl:M0805
- added R22, R23: 8k2, rcl:M0805
- added R26: 180, rcl:M0805
- added R30: 0.33r, rcl:M1206
- added R31: 470, rcl:M0805
- added R32: 1k, rcl:M0805
- added R34, R35: 47k, rcl:0207/10
- added R36: 1k, rcl:0207/10
- added R37: 30k, rcl:0207/10
- added R38, R39, R40: 15k, rcl:0207/10
- added R41, R42: 220, rcl:0207/10
- added R43: 10k, rcl:0207/10
- added U$19, U$21, U$22: (no value), ie13:EE15
- added VT10, VT8: BJT_NPN_TO-92_CBE, m_transistor:TO92
- added VT11, VT9: BJT_PNP_TO-92_CBE, m_transistor:TO92
- added VT2, VT7: (no value), m_transistor:DPACK
- added VT3, VT5: КТ3102, transistor-npn:TO92-EBC
- moved R18 238.7 mm to (141.6, 126.4), flipped to the bottom
- moved V6 61.3 mm to (-80.6, 111.1)
- moved U$7 43.9 mm to (128.9, 81.3)
- moved U$9 39.2 mm to (120.7, 167.0)
Connections:
- new net -24V: C30.1, D12.A
- new net N$100: IV3A.2, R.1
- new net N$101: C28.+, R37.2, R38.2, VT10.3, VT11.3
- new net N$102: C25.2, C26.1, DA4.9, R34.1, R35.2, R36.1
- new net N$103: C25.1, R34.2, VT9.2
- new net N$104: C26.2, R35.1, VT8.2
- new net N$105: C30.2, D12.C, R41.1, R42.2, R43.2
- new net N$106: C28.-, R41.2
- new net N$107: C29.-, R42.1
- new net N$109: DA4.4, R37.1, R39.2, R40.1
- new net N$110: C27.1, DA4.3, R38.1
- new net N$28: C16.1, L4.2, VT5.C
- new net N$69: R19.1, VT2.G
- new net N$70: C203.2, DA2.2, DA2.4, VT2.D
- new net N$71: C15.2, L6.1, VT3.C
- new net N$72: R20.1, R22.1, VT5.B
- new net N$73: R21.1, R23.1, VT3.B
- new net N$74: DA1.8, R26.2
- new net N$75: L4.1, L6.2, R22.2, R23.2
- new net N$76: C16.2, R21.2
- new net N$78: DA1.7, L8.1, R26.1, R30.2
- new net N$80: C15.1, R20.2
- new net N$83: VT10.2, VT11.2, VT8.1, VT9.1
- new net N$87: C19.1, DA1.3
- new net N$89: C24.1, DA1.5, R31.1, R32.2
- new net N$90: D10.A, L9.2
- new net N$95: R33.1, VT7.G
- new net N$96: C20.2, C22.-, D11.C, IV1.1, IV2.1, IV3.1, IV3A.1, IV6.1
- new net N$97: D10.C, R31.2
- new net N$99: C20.1, C22.+, DA1.1, IV1.2, IV2.2, IV3.2, IV6.2, L8.2, L9.1, R.2
- new net V+: DA4.11, R36.2, R40.2, VT10.1, VT9.3
- net +3V3: now also C21.1, C23.+, DA1.6, R30.1
- net GND: now also C19.2, C21.2, C23.-, C24.2, C27.2, C29.+, D11.A, DA1.2, DA1.4, DA4.2, DA4.6, R19.2, R32.1, R33.2, R39.1, R43.1, VT11.1, VT2.S, VT3.E, VT5.E, VT7.S, VT8.3; no longer C203.2, DA2.2, DA2.4
Routing:
- net V+: track 0.00 -> 21.3 mm
- net N$83: track 0.00 -> 15.7 mm
- net N$103: track 0.00 -> 11.9 mm
- net N$104: track 0.00 -> 11.3 mm
- net N$102: track 0.00 -> 9.90 mm
- net GND: track 34.1 -> 44.0 mm
- net N$101: track 0.00 -> 7.24 mm

Commit message: .
Parts:
- added C31: 100m, rcl:E2-5
- added R46: 1k, rcl:M0805
- added R47: 270, rcl:M0805
- added U$24: TRAN_EE16, ie13:EE16
- added VT14, VT15: BC847, m_transistor:SOT23
- R36, R39: device rcl:0207/10 -> rcl:M0805
- moved R38 46.6 mm to (-79.4, -5.71)
- moved R41 42.3 mm to (-72.4, 1.91), turned to 90 degrees
- moved R42 40.6 mm to (-76.8, 0.64), turned to 270 degrees
- moved R37 35.3 mm to (-79.4, 18.4)
- moved C30 28.9 mm to (-83.8, -29.2)
- moved D12 28.4 mm to (-83.2, -20.3), turned to 180 degrees
- moved R43 28.4 mm to (-83.2, -15.9)
- moved R40 24.5 mm to (-89.5, 22.2), turned to 180 degrees
- moved R39 18.5 mm to (-117.5, 8.26), flipped to the bottom, turned to 270 degrees
- moved DA4 14.5 mm to (-117.5, 8.26)
- moved C27 14.3 mm to (-121.3, 0.64)
- moved R36 10.9 mm to (-114.3, 15.2), flipped to the bottom, turned to 0 degrees
- moved R34 2.01 mm to (-103.5, 18.4)
Connections:
- new net N$116: U$24.1, VT15.3
- new net N$117: U$24.3, VT14.3
- new net N$118: U$24.2, VT14.1
- new net N$119: U$24.6, VT15.1
- new net N$120: R46.1, U$24.5
- new net N$121: C31.-, R46.2, R47.2, U$24.4
- net GND: now also C31.+, R47.1, VT14.2, VT15.2
Routing:
- net GND: track 44.0 -> 71.1 mm
- net N$119: track 0.00 -> 25.2 mm
- net N$102: track 9.90 -> 26.8 mm
- net V+: track 21.3 -> 38.1 mm
- net N$118: track 0.00 -> 7.77 mm
- net N$116: track 0.00 -> 5.08 mm
- net N$110: track 0.00 -> 3.81 mm
- net N$109: track 0.00 -> 2.86 mm
- net N$117: track 0.00 -> 2.34 mm

Commit message: .
Parts:
- removed U$19, U$21: (no value), ie13:EE15
- removed U$9: (no value), ie13:1420
- added R44: 0, rcl:R1206
- C31: device rcl:E2-5 -> rcl:SANYO-OSCON_SMD_A5
- U$7: value (none) -> TRAN_EE16; device ie13:1420 -> ie13:EE16
- moved U$24 319.7 mm to (86.0, 145.7), turned to 90 degrees
- moved R46 308.0 mm to (77.5, 145.3), flipped to the bottom, turned to 270 degrees
- moved VT14 299.2 mm to (74.8, 143.1), flipped to the bottom, turned to 0 degrees
- moved C31 297.4 mm to (69.3, 139.2), flipped to the bottom, turned to 180 degrees
- moved R47 296.9 mm to (68.3, 142.4), flipped to the bottom, turned to 0 degrees
- moved VT15 293.6 mm to (74.6, 139.1), flipped to the bottom, turned to 0 degrees
- moved U$7 42.9 mm to (86.0, 82.0), turned to 90 degrees
- moved DD4 15.3 mm to (52.3, 146.2)
- moved JP10 14.0 mm to (52.7, 139.3)
Connections:
- removed net +3V3: C201.+, C202.1, C21.1, C23.+, C5.1, DA1.6, DA2.6, DA3.6, JP19.1, L1.2, R1B1.1, R201.1, R30.1, U$13.4, U$13.5
- removed net N$120: R46.1, U$24.5
- new net +3V7: C201.+, C202.1, C21.1, C23.+, C5.1, DA1.6, DA2.6, DA3.6, JP19.1, L1.2, R1B1.1, R201.1, R30.1, R46.1, U$13.4, U$13.5, U$24.3
- new net HE3: V3.7
- new net HK3: V3.8
- new net N$77: R44.1, VT14.2
- net GND: now also R44.2; no longer VT14.2
- net N$117: now also U$24.2; no longer U$24.3
- net N$118: now also U$24.5; no longer U$24.2
Routing:
- net N$121: track 0.00 -> 33.5 mm
- net N$119: track 25.2 -> 4.90 mm
- net N$116: track 5.08 -> 20.5 mm
- net N$117: track 2.34 -> 9.60 mm
- net N$118: track 7.77 -> 4.40 mm
- net N$77: track 0.00 -> 3.36 mm
- net +3V7: track 0.00 -> 2.83 mm
- net GND: track 71.1 -> 73.0 mm

Commit message: >d
Parts:
- removed C15, C16: 22n, rcl:C1206
- removed C17: 10u/100V, rcl:TT5D9L
- removed C18: 510, resistor:C0805K
- removed C19: 120, rcl:C0805
- removed C20, C21, C24: 100n, rcl:C0805
- removed C22: 100m, rcl:E2,5-5
- removed C23: 470m, rcl:E3,5-8
- removed C25, C26: 33, rcl:C025-025X050
- removed C27: 2n2, rcl:C025-025X050
- removed C28, C29: 100m, rcl:E2-5
- removed C30: 1m, rcl:C025-025X050
- removed C31: 100m, rcl:SANYO-OSCON_SMD_A5
- removed D10, D11: (no value), diode:SOD80C
- removed D12: (no value), diode:DO34Z7
- removed DA1: MC34063AD, mc34063-2:SOIC8
- removed DA3: MC34063AD, mc34063:SOIC8
- removed DA4: LM311,К554СА3KY, IC:DIL14
- removed IV1, IV2, IV3, IV6: 24r, rcl:M0805
- removed IV3A: 17r, rcl:M0805
- removed JP10: (no value), Разъёмы штырьковые 2.54мм:1X07
- removed L2, L3: (no value), rcl:IR-2
- removed L4, L6, L7: (no value), rcl:L3225M
- removed L5: 150uH, rcl:0204/7
- removed L8, L9: 50mkhn, rcl:TFI0305
- removed R: (no value), rcl:M0805
- removed R1B1, R1B2: 0.22, resistor:R1206
- removed R22, R23: 8k2, rcl:M0805
- removed R24: 15k, rcl:R0805
- removed R25, R27: 1k, rcl:R0805
- removed R26: 180, rcl:M0805
- removed R28: 330, rcl:R0805
- removed R29: 1k(330), rcl:R0805
- removed R30: 0.33r, rcl:M1206
- removed R31: 470, rcl:M0805
- removed R32, R36, R46: 1k, rcl:M0805
- removed R33: 100k, rcl:M0805
- removed R34, R35: 47k, rcl:0207/10
- removed R37: 30k, rcl:0207/10
- removed R38, R40: 15k, rcl:0207/10
- removed R39: 15k, rcl:M0805
- removed R41, R42: 220, rcl:0207/10
- removed R43: 10k, rcl:0207/10
- removed R44: 0, rcl:R1206
- removed R47: 270, rcl:M0805
- removed T3, T4: (no value), transistor:TO126
- removed U$22: (no value), ie13:EE15
- removed U$24: TRAN_EE16, ie13:EE16
- removed V6: ИВ-6, vfd:CON_VFD
- removed VD3: FR207, diode:DO41-10
- removed VD4: 1N4148, diode:SOD80C
- removed VT10, VT8: BJT_NPN_TO-92_CBE, m_transistor:TO92
- removed VT11, VT9: BJT_PNP_TO-92_CBE, m_transistor:TO92
- removed VT14, VT15: BC847, m_transistor:SOT23
- removed VT4: КТ3107, transistor-pnp:TO92-CBE
- removed VT5, VT6: КТ3102, transistor-npn:TO92-EBC
- removed VT7: (no value), m_transistor:DPACK
- added JP1: (no value), Разъёмы штырьковые 2.54мм:1X07
- added T19: (no value), transistor:TO92-ECB
- added U$9: MOD_TP4056, TP4056+mod:MOD_03962A
- C14: value 10n -> (none); device rcl:C0805 -> rcl:C1206
- C5: value (none) -> 10m; device rcl:C1206 -> rcl:SANYO-OSCON_SMD_A5
- R17: value 10k -> (none); device rcl:M0805 -> rcl:RTRIM3296W
- R18: value 10k -> 68k
- R20: value 56k -> 2k2
- R21: value 56k -> (none)
- R6: value (none) -> 1k; device rcl:RTRIM3296W -> rcl:M0805
- R7: value 68k -> 270
- R8: value 2k2 -> 0; device rcl:M0805 -> rcl:M1206
- T1: value (none) -> TRAN_EE16; device transistor:TO92-ECB -> ie13:EE16
- VT1: value (none) -> BC847; device m_transistor:DPACK -> m_transistor:SOT23
- VT3: value КТ3102 -> BC847; device transistor-npn:TO92-EBC -> m_transistor:SOT23
- moved R20 223.3 mm to (19.1, 219.7), flipped to the bottom, turned to 180 degrees
- moved C10 213.3 mm to (172.1, 141.6)
- moved C4 213.3 mm to (197.5, 158.8)
- moved C7 213.3 mm to (156.2, 166.4)
- moved D6 213.3 mm to (156.2, 170.8)
- moved D7 213.3 mm to (156.2, 156.8)
- moved R13 213.3 mm to (148.0, 144.1)
- moved R14 213.3 mm to (160.0, 141.6)
- moved R15 213.3 mm to (179.7, 142.2)
- moved R16 213.3 mm to (165.7, 170.8)
- moved R9 213.3 mm to (156.2, 160.0)
- moved C8 213.3 mm to (156.8, 153.0)
- moved C9 213.3 mm to (176.5, 163.8)
- moved D8 213.3 mm to (155.6, 144.8)
- moved D9 213.3 mm to (167.0, 141.6)
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Connections:
- removed net -24V: C30.1, D12.A
- removed net N$100: IV3A.2, R.1
- removed net N$101: C28.+, R37.2, R38.2, VT10.3, VT11.3
- removed net N$102: C25.2, C26.1, DA4.9, R34.1, R35.2, R36.1
- removed net N$103: C25.1, R34.2, VT9.2
- removed net N$104: C26.2, R35.1, VT8.2
- removed net N$105: C30.2, D12.C, R41.1, R42.2, R43.2
- removed net N$106: C28.-, R41.2
- removed net N$107: C29.-, R42.1
- removed net N$109: DA4.4, R37.1, R39.2, R40.1
- removed net N$110: C27.1, DA4.3, R38.1
- removed net N$34 (its old number): DD4.4, JP10.4
- removed net N$46: T3.2, T4.3
- removed net N$71: C15.2, L6.1, VT3.C
- removed net N$72: R20.1, R22.1, VT5.B
- removed net N$73: R21.1, R23.1, VT3.B
- removed net N$74: DA1.8, R26.2
- removed net N$75: L4.1, L6.2, R22.2, R23.2
- removed net N$76: C16.2, R21.2
- removed net N$77: R44.1, VT14.2
- removed net N$78: DA1.7, L8.1, R26.1, R30.2
- removed net N$79: DA3.2, R27.1, R28.1, R28.2, R29.2, VD4.A, VT4.B, VT6.B
- removed net N$80: C15.1, R20.2
- removed net N$81: C14.1, R17.1, T3.3
- removed net N$82: C14.2, L2.1, T4.2
- removed net N$83: VT10.2, VT11.2, VT8.1, VT9.1
- removed net N$85: L3.1
- removed net N$86: L3.2
- removed net N$87: C19.1, DA1.3
- removed net N$88: L5.2, VD3.A, VT1.D
- removed net N$89: C24.1, DA1.5, R31.1, R32.2
- removed net N$90: D10.A, L9.2
- removed net N$91: DA3.5, R24.1, R25.2
- removed net N$92: C17.+, R24.2, VD3.C
- removed net N$93: R27.2, VD4.C, VT1.G, VT4.E, VT6.E
- removed net N$94: DA3.7, L5.1, R1B1.2
- removed net N$95: R33.1, VT7.G
- removed net N$96: C20.2, C22.-, D11.C, IV1.1, IV2.1, IV3.1, IV3A.1, IV6.1
- removed net N$97: D10.C, R31.2
- removed net N$98: C18.1, DA3.3
- removed net N$99: C20.1, C22.+, DA1.1, IV1.2, IV2.2, IV3.2, IV6.2, L8.2, L9.1, R.2
- removed net V+: DA4.11, R36.2, R40.2, VT10.1, VT9.3
- removed net VCC/2: R17.2, T4.1
- new net +3V3: C6.1, JP19.1, L1.2, U$13.4, U$13.5
- new net N$27: C5.+, R7.1, R8.2, VT1.2, VT3.2
- new net SD: R21.2, V3.9
- net +30V: now also R21.1; no longer R18.2
- net +3V7: now also R6.1, T1.5; no longer C21.1, C23.+, C5.1, DA1.6, DA3.6, JP19.1, L1.2, R1B1.1, R30.1, R46.1, U$13.4, U$13.5, U$24.3
- net GND: now also C14.2, R20.1; no longer C17.-, C18.2, C19.2, C21.2, C23.-, C24.2, C27.2, C29.+, C31.+, C5.2, D11.A, DA1.2, DA1.4, DA3.4, DA4.2, DA4.6, L2.2, R25.1, R29.1, R32.1, R33.2, R39.1, R43.1, R44.2, R47.1, R8.1, T3.1, VT1.S, VT11.1, VT15.2, VT3.E, VT4.C, VT5.E, VT7.S, VT8.3
- net N$116: now also T1.1, VT1.3; no longer U$24.1, VT15.3
- net N$117: now also T1.3, VT3.3; no longer U$24.2, VT14.3
- net N$118: now also T1.2, VT3.1; no longer U$24.5, VT14.1
- net N$119: now also T1.6, VT1.1; no longer U$24.6, VT15.1
- net N$121: now also C5.-, R6.2, R7.2, T1.4; no longer C31.-, R46.2, R47.2, U$24.4
- net N$17: now also T19.E; no longer T1.E
- net N$26: now also DD4.4, JP1.4; no longer DA3.1, DA3.8, R18.1, R1B2.1, R1B2.2, VT6.C
- net N$28: now also R8.1, VT2.D; no longer C16.1, L4.2, VT5.C
- net N$31: now also JP1.1; no longer JP10.1
- net N$32: now also JP1.2; no longer JP10.2
- net N$33: now also JP1.3; no longer JP10.3
- net N$36: now also T19.B; no longer T1.B
- net N$43: now also R17.3, R18.1; no longer R6.3, R7.1
- net N$44: now also R17.2; no longer R6.2
- net N$45: now also R17.1, R20.2; no longer R6.1, R8.2
- net N$65: now also JP1.5; no longer JP10.5
- net N$67: now also JP1.6; no longer JP10.6
- net N$68: now also JP1.7; no longer JP10.7
- net N$70: no longer VT2.D
- net VCC: now also C14.1, R18.2, T19.C; no longer C6.1, R7.2, T1.C
Routing:
- net GND: track 73.0 -> 34.1 mm
- net V+: track 38.1 -> 0.00 mm
- net N$102: track 26.8 -> 0.00 mm
- net N$121: track 33.5 -> 10.3 mm
- net N$119: track 4.90 -> 26.1 mm
- net N$116: track 20.5 -> 4.64 mm
- net N$83: track 15.7 -> 0.00 mm
- net N$103: track 12.2 -> 0.00 mm
- net N$104: track 11.3 -> 0.00 mm
- net N$27: track 0.00 -> 8.90 mm
- net N$101: track 7.24 -> 0.00 mm
- net N$117: track 9.60 -> 4.13 mm
- net N$110: track 3.81 -> 0.00 mm
- net N$77: track 3.36 -> 0.00 mm
- net N$109: track 2.86 -> 0.00 mm
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
Commit message: .
Parts:
- S3, S4.1, S5: device switch-omron:B3F-10XX -> switch:SKHMPXE010
- moved S5 88.9 mm to (85.7, 176.5), flipped to the bottom
- moved S4.1 87.2 mm to (73.0, 175.9), flipped to the bottom
- moved S3 56.5 mm to (58.4, 176.5), flipped to the bottom
- moved S1 0.63 mm to (45.7, 175.3)
Connections:
- net N$11: now also S5.1, S5.2; no longer S5.3, S5.4
- net N$12: now also S3.1, S3.2; no longer S3.3, S3.4
- net N$13: now also S4.1.1, S4.1.2; no longer S4.1.3, S4.1.4
- net N$15: now also S3.3, S3.4, S4.1.3, S4.1.4; no longer S3.1, S3.2, S4.1.1, S4.1.2
- net VCC: now also S5.3, S5.4; no longer S5.1, S5.2
Changed lines of the file:
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@@
 <element name="R3" library="rcl" package="M0805" value="10k" x="40.005" y="164.465" rot="MR180"/>
 <element name="C3" library="rcl" package="C0805" value="10n" x="40.005" y="167.64" rot="MR0"/>
-<element name="S3" library="switch-omron" package="B3F-10XX" value="УЧ" x="3.81" y="161.925">
-<attribute name="OC_NEWARK" value="36M3542" x="3.81" y="161.925" size="1.778" layer="27" display="off"/>
-<attribute name="MPN" value="B3F-1000" x="3.81" y="161.925" size="1.778" layer="27" display="off"/>
-<attribute name="MF" value="" x="3.81" y="161.925" size="1.778" layer="27" display="off"/>
-<attribute name="OC_FARNELL" value="176432" x="3.81" y="161.925" size="1.778" layer="27" display="off"/>
-</element>
-<element name="S4.1" library="switch-omron" package="B3F-10XX" value="УБ" x="-13.335" y="163.83">
-<attribute name="OC_NEWARK" value="36M3542" x="-13.335" y="163.83" size="1.778" layer="27" display="off"/>
-<attribute name="MPN" value="B3F-1000" x="-13.335" y="163.83" size="1.778" layer="27" display="off"/>
-<attribute name="MF" value="" x="-13.335" y="163.83" size="1.778" layer="27" display="off"/>
-<attribute name="OC_FARNELL" value="176432" x="-13.335" y="163.83" size="1.778" layer="27" display="off"/>
-</element>
 <element name="DD3" library="К176" package="DIL16B" value="К176ИД2,ИД3" x="64.77" y="149.86" rot="R180"/>
 <element name="R4" library="rcl" package="M0805" value="100k" x="58.42" y="161.925" rot="MR180"/>
-<element name="S5" library="switch-omron" package="B3F-10XX" value="УЧ" x="-3.175" y="175.26">
-<attribute name="OC_NEWARK" value="36M3542" x="-3.175" y="175.26" size="1.778" layer="27" display="off"/>
-<attribute name="MPN" value="B3F-1000" x="-3.175" y="175.26" size="1.778" layer="27" display="off"/>
-<attribute name="MF" value="" x="-3.175" y="175.26" size="1.778" layer="27" display="off"/>
-<attribute name="OC_FARNELL" value="176432" x="-3.175" y="175.26" size="1.778" layer="27" display="off"/>
-</element>
 <element name="T19" library="transistor" package="TO92-ECB" value="" x="210.82" y="154.305" rot="R270"/>
 <element name="T2" library="transistor" package="TO92-BCE" value="" x="207.01" y="156.21" rot="R270"/>
@@
 <element name="V4" library="vfd" package="CON_VFD" value="ИВ-6" x="73.66" y="229.87"/>
 <element name="V5" library="vfd" package="CON_VFD" value="ИВ-6" x="86.36" y="229.87"/>
-<element name="S1" library="switch" package="SKHMPXE010" value="Ч" x="46.355" y="175.26" rot="MR0"/>
+<element name="S1" library="switch" package="SKHMPXE010" value="Ч" x="45.72" y="175.26" rot="MR0"/>
 <element name="S2" library="switch" package="SKHMPXE010" value="М" x="31.75" y="175.26" rot="MR0"/>
 <element name="VT2" library="m_transistor" package="DPACK" value="" x="61.595" y="222.885" rot="MR90"/>
@@
 <element name="U$9" library="TP4056+mod" package="MOD_03962A" value="MOD_TP4056" x="-22.225" y="224.79" rot="MR270"/>
 <element name="R21" library="rcl" package="M0805" value="" x="60.325" y="237.49" rot="MR0"/>
+<element name="S3" library="switch" package="SKHMPXE010" value="УЧ" x="58.42" y="176.53" rot="MR0"/>
+<element name="S4.1" library="switch" package="SKHMPXE010" value="УБ" x="73.025" y="175.895" rot="MR0"/>
+<element name="S5" library="switch" package="SKHMPXE010" value="УЧ" x="85.725" y="176.53" rot="MR0"/>
 </elements>
 <signals>
@@
 <contactref element="T19" pad="C"/>
 <contactref element="DD2" pad="2"/>
-<contactref element="S5" pad="2"/>
-<contactref element="S5" pad="1"/>
 <contactref element="J1" pad="1"/>
 <wire x1="73.66" y1="146.05" x2="73.66" y2="147.955" width="0.4064" layer="16"/>
@@
 <contactref element="D5" pad="C"/>
 <contactref element="C14" pad="1"/>
+<contactref element="S5" pad="4"/>
+<contactref element="S5" pad="3"/>
 <wire x1="18.415" y1="229.55" x2="18.12" y2="234.95" width="0" layer="19" extent="16-16"/>
 <wire x1="23.495" y1="219.205" x2="18.415" y2="229.55" width="0" layer="19" extent="16-16"/>
-<wire x1="0.0762" y1="177.5206" x2="23.495" y2="219.205" width="0" layer="19" extent="16-16"/>
-<wire x1="-6.4262" y1="177.5206" x2="0.0762" y2="177.5206" width="0" layer="19" extent="1-1"/>
-<wire x1="37.465" y1="150.815" x2="0.0762" y2="177.5206" width="0" layer="19" extent="16-16"/>
+<wire x1="71.12" y1="168.275" x2="23.495" y2="219.205" width="0" layer="19" extent="16-16"/>
+<wire x1="64.45" y1="161.925" x2="71.12" y2="165.1" width="0" layer="19" extent="16-16"/>
+<wire x1="81.525" y1="174.28" x2="75.565" y2="168.275" width="0" layer="19" extent="16-16"/>
+<wire x1="89.925" y1="174.28" x2="81.525" y2="174.28" width="0" layer="19" extent="16-16"/>
+<wire x1="37.465" y1="150.815" x2="62.36" y2="151.13" width="0" layer="19" extent="16-16"/>
 <wire x1="35.56" y1="143.51" x2="37.465" y2="150.815" width="0" layer="19" extent="16-16"/>
-<wire x1="62.36" y1="151.13" x2="37.465" y2="150.815" width="0" layer="19" extent="16-16"/>
-<wire x1="64.45" y1="161.925" x2="71.12" y2="165.1" width="0" layer="19" extent="16-16"/>
-<wire x1="210.82" y1="154.305" x2="75.565" y2="157.48" width="0" layer="19" extent="16-16"/>
+<wire x1="210.82" y1="154.305" x2="89.925" y2="174.28" width="0" layer="19" extent="16-16"/>
 </signal>
 <signal name="N$1">
@@
 <contactref element="S1" pad="1"/>
 <contactref element="S1" pad="2"/>
-<wire x1="42.155" y1="177.51" x2="50.555" y2="177.51" width="0" layer="19" extent="16-16"/>
-<wire x1="46.355" y1="154.1" x2="50.555" y2="177.51" width="0" layer="19" extent="16-16"/>
+<wire x1="41.52" y1="177.51" x2="49.92" y2="177.51" width="0" layer="19" extent="16-16"/>
+<wire x1="46.355" y1="154.1" x2="41.52" y2="177.51" width="0" layer="19" extent="16-16"/>
 </signal>
 <signal name="N$4">
@@
 <signal name="N$12">
 <contactref element="D4" pad="A"/>
-<contactref element="S3" pad="3"/>
-<contactref element="S3" pad="4"/>
 <contactref element="S1" pad="4"/>
 <contactref element="S1" pad="3"/>
 <contactref element="S2" pad="3"/>
 <contactref element="S2" pad="4"/>
-<wire x1="42.155" y1="173.01" x2="50.555" y2="173.01" width="0" layer="19" extent="16-16"/>
-<wire x1="35.95" y1="173.01" x2="42.155" y2="173.01" width="0" layer="19" extent="16-16"/>
+<contactref element="S3" pad="1"/>
+<contactref element="S3" pad="2"/>
+<wire x1="54.22" y1="178.78" x2="62.62" y2="178.78" width="0" layer="19" extent="16-16"/>
+<wire x1="49.92" y1="173.01" x2="54.22" y2="178.78" width="0" layer="19" extent="16-16"/>
+<wire x1="41.52" y1="173.01" x2="49.92" y2="173.01" width="0" layer="19" extent="16-16"/>
+<wire x1="35.95" y1="173.01" x2="41.52" y2="173.01" width="0" layer="19" extent="16-16"/>
 <wire x1="35.355" y1="167.64" x2="35.95" y2="173.01" width="0" layer="19" extent="16-16"/>
 <wire x1="27.55" y1="173.01" x2="35.95" y2="173.01" width="0" layer="19" extent="16-16"/>
-<wire x1="7.0612" y1="159.6644" x2="27.55" y2="173.01" width="0" layer="19" extent="16-16"/>
-<wire x1="0.5588" y1="159.6644" x2="7.0612" y2="159.6644" width="0" layer="19" extent="1-1"/>
 </signal>
 <signal name="N$13">
 <contactref element="D4" pad="C"/>
 <contactref element="D3" pad="C"/>
-<contactref element="S4.1" pad="4"/>
-<contactref element="S4.1" pad="3"/>
+<contactref element="S4.1" pad="2"/>
+<contactref element="S4.1" pad="1"/>
+<wire x1="77.225" y1="178.145" x2="68.825" y2="178.145" width="0" layer="19" extent="16-16"/>
+<wire x1="46.355" y1="165.53" x2="68.825" y2="178.145" width="0" layer="19" extent="16-16"/>
 <wire x1="31.955" y1="167.64" x2="46.355" y2="165.53" width="0" layer="19" extent="16-16"/>
-<wire x1="-10.0838" y1="161.5694" x2="31.955" y2="167.64" width="0" layer="19" extent="16-16"/>
-<wire x1="-16.5862" y1="161.5694" x2="-10.0838" y2="161.5694" width="0" layer="19" extent="1-1"/>
 </signal>
 <signal name="N$15">
-<contactref element="S3" pad="1"/>
-<contactref element="S3" pad="2"/>
-<contactref element="S4.1" pad="1"/>
-<contactref element="S4.1" pad="2"/>
 <contactref element="C3" pad="1"/>
 <contactref element="R3" pad="2"/>
 <contactref element="DD2" pad="11"/>
-<wire x1="40.955" y1="164.465" x2="60.96" y2="157.48" width="0" layer="19" extent="16-16"/>
-<wire x1="40.955" y1="167.64" x2="40.955" y2="164.465" width="0" layer="19" extent="16-16"/>
-<wire x1="7.0612" y1="164.1856" x2="40.955" y2="164.465" width="0" layer="19" extent="16-16"/>
-<wire x1="0.5588" y1="164.1856" x2="7.0612" y2="164.1856" width="0" layer="19" extent="1-1"/>
-<wire x1="-10.0838" y1="166.0906" x2="0.5588" y2="164.1856" width="0" layer="19" extent="1-1"/>
-<wire x1="-16.5862" y1="166.0906" x2="-10.0838" y2="166.0906" width="0" layer="19" extent="1-1"/>
+<contactref element="S3" pad="4"/>
+<contactref element="S3" pad="3"/>
+<contactref element="S4.1" pad="4"/>
+<contactref element="S4.1" pad="3"/>
+<wire x1="62.62" y1="174.28" x2="68.825" y2="173.645" width="0" layer="19" extent="16-16"/>
+<wire x1="54.22" y1="174.28" x2="62.62" y2="174.28" width="0" layer="19" extent="16-16"/>
+<wire x1="77.225" y1="173.645" x2="68.825" y2="173.645" width="0" layer="19" extent="16-16"/>
+<wire x1="60.96" y1="157.48" x2="54.22" y2="174.28" width="0" layer="19" extent="16-16"/>
+<wire x1="40.955" y1="167.64" x2="54.22" y2="174.28" width="0" layer="19" extent="16-16"/>
+<wire x1="40.955" y1="164.465" x2="40.955" y2="167.64" width="0" layer="19" extent="16-16"/>
 </signal>
 <signal name="N$5">
@@
 <contactref element="R4" pad="2"/>
 <contactref element="DD2" pad="6"/>
-<contactref element="S5" pad="4"/>
-<contactref element="S5" pad="3"/>
+<contactref element="S5" pad="1"/>
+<contactref element="S5" pad="2"/>
 <wire x1="59.37" y1="161.925" x2="60.96" y2="165.1" width="0" layer="19" extent="16-16"/>
-<wire x1="0.0762" y1="172.9994" x2="59.37" y2="161.925" width="0" layer="19" extent="16-16"/>
-<wire x1="-6.4262" y1="172.9994" x2="0.0762" y2="172.9994" width="0" layer="19" extent="1-1"/>
+<wire x1="81.525" y1="178.78" x2="60.96" y2="165.1" width="0" layer="19" extent="16-16"/>
+<wire x1="89.925" y1="178.78" x2="81.525" y2="178.78" width="0" layer="19" extent="16-16"/>
 </signal>
 <signal name="N$14">
