File: K176IE13.brd (EAGLE design)
At the start: 99 parts, among them T1 TRAN_EE16

Commit message: b
Parts:
- removed U$1: (no value), vfd:IV-3A_H
- removed U$3: (no value), vfd:IV-6_H
- removed V3: ИВ-3А, vfd:CON_VFD
- U$4: value (none) -> IV-3T_VIXC; device vfd:IV-6_H -> vfd:IV-3A_VIXC
- U$5: device vfd:IV-6_H -> vfd:CON_VFD_SCH
- V1, V5: device vfd:CON_VFD -> vfd:IV-6_VIXC
- V2: value ИВ-6 -> IV-6_T_VIXL; device vfd:CON_VFD -> vfd:IV-6_VIXL
- moved V1 223.7 mm to (-25.4, 14.6)
- moved V2 223.7 mm to (-12.7, 14.6)
- moved V5 223.7 mm to (25.4, 14.6)
- moved JP1 213.4 mm to (2.54, 2.54)
- moved DD4 211.0 mm to (54.0, 3.03)
- moved U$4 206.9 mm to (0.00, 14.6), turned to 0 degrees
- moved U$12 204.9 mm to (-0.00, -0.63)
- moved C1 204.3 mm to (-31.1, -40.0)
- moved C12 204.3 mm to (2.54, -33.0)
- moved C2 204.3 mm to (-29.2, -30.5)
- moved C204 204.3 mm to (102.9, 6.99)
- moved C205 204.3 mm to (109.2, 0.64)
- moved C4 204.3 mm to (136.5, -36.2)
- moved C5 204.3 mm to (9.52, 19.7)
- moved C7 204.3 mm to (95.2, -28.6)
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Connections:
- net HE3: now also U$4.7; no longer V3.7
- net HK3: now also U$4.8; no longer V3.8
- net SD: now also U$4.9; no longer V3.9
Routing:
- net A: track 68.7 -> 64.2 mm
- net E: track 68.6 -> 64.1 mm
- net HE: track 66.1 -> 62.3 mm
- net D: track 66.0 -> 62.2 mm
- net F: track 65.2 -> 61.6 mm
- net HK: track 63.6 -> 60.4 mm
- net G: track 63.5 -> 60.3 mm
- net C: track 61.0 -> 58.4 mm
- net B: track 58.4 -> 56.5 mm

Commit message: .
Parts:
- removed U$12: (no value), ie13:1865
- removed U$2: (no value), vfd:IV-6_H
- removed U$4: IV-3T_VIXC, vfd:IV-3A_VIXC
- added V3: ИВ-3А, vfd:IV-3A_VIXC
- V2: value IV-6_T_VIXL -> ИВ-6
- V4: device vfd:CON_VFD -> vfd:IV-6_VIXR
- moved DD50 59.8 mm to (60.3, -24.1), turned to 0 degrees
- moved JP19 55.2 mm to (21.6, 23.5)
- moved DD4 53.6 mm to (0.62, -2.68)
- moved L1 42.5 mm to (17.8, 23.5)
- moved V4 41.3 mm to (12.7, -6.35)
- moved U$9 37.3 mm to (-58.4, 1.91)
- moved U$13 34.2 mm to (14.0, 23.5)
- moved C6 30.5 mm to (13.3, 26.0), turned to 180 degrees
- moved R17 28.4 mm to (5.08, 31.8)
- moved R18 23.9 mm to (4.44, 23.5)
- moved C14 23.9 mm to (8.89, 24.8)
- moved R20 23.6 mm to (6.98, 24.8)
- moved R21 22.0 mm to (3.81, 21.0)
- moved T1 21.8 mm to (24.8, -3.17)
- moved R8 21.7 mm to (12.1, 3.81)
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Connections:
- net HE3: now also V3.7; no longer U$4.7
- net HK3: now also V3.8; no longer U$4.8
- net SD: now also V3.9; no longer U$4.9
Routing:
- net N$121: track 10.3 -> 17.0 mm
- net A: track 64.2 -> 68.7 mm
- net E: track 64.1 -> 68.6 mm
- net HE: track 62.3 -> 66.1 mm
- net D: track 62.2 -> 66.0 mm
- net F: track 61.6 -> 65.2 mm
- net N$27: track 8.90 -> 12.4 mm
- net HK: track 60.4 -> 63.6 mm
- net G: track 60.3 -> 63.5 mm
- net N$119: track 26.1 -> 28.9 mm
- net C: track 58.4 -> 61.0 mm
- net B: track 56.5 -> 58.4 mm

Commit message: .
Parts:
- removed JP19: (no value), Разъёмы штырьковые 2.54мм:1X02
- removed JP6, JP7: (no value), Разъёмы штырьковые 2.54мм:1X01
- removed U$7: TRAN_EE16, ie13:EE16
- added JP2: (no value), Разъёмы штырьковые 2.54мм:1X04
- added R22, R23: (no value), rcl:M0805
- added T3: TRAN_EE16, ie13:EE16
- added XBAT: (no value), Разъёмы штырьковые 2.54мм:1X02
- DD1, DD2: device К176:DIL16 -> К176:DIL16B
- moved C10 66.8 mm to (52.7, -21.0), turned to 180 degrees
- moved R15 64.6 mm to (68.6, -12.1)
- moved D9 58.0 mm to (63.5, -14.0)
- moved T19 50.3 mm to (104.1, -19.7), turned to 90 degrees
- moved C9 46.2 mm to (71.1, -18.4), turned to 0 degrees
- moved D8 44.1 mm to (56.5, -27.9)
- moved R9 43.3 mm to (52.1, -38.7)
- moved R11 43.2 mm to (69.2, -26.0), turned to 270 degrees
- moved R13 42.6 mm to (51.4, -27.3)
- moved R10 41.4 mm to (65.4, -19.1), turned to 180 degrees
- moved R14 40.4 mm to (62.2, -36.8), turned to 270 degrees
- moved D7 39.5 mm to (55.9, -35.6)
- moved T2 37.8 mm to (113.0, -20.3)
- moved R5 36.9 mm to (109.2, -19.0)
- moved U$6 36.6 mm to (108.6, -31.1)
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Connections:
- new net N$46: U$9.P2+B, XBAT.1
- new net N$71: R23.1
- new net N$72: DD6.4, JP2.1
- new net N$73: DD6.5, JP2.2
- new net N$74: DD6.6, JP2.3
- new net N$75: DD6.7, JP2.4
- net +3V3: now also U$9.P2+OUT; no longer JP19.1
- net GND: now also C203.2, DA2.2, DA2.4, U$9.P2-OUT; no longer JP19.2
- net HE3: now also R22.2
- net HK3: now also R23.2
- net N$47: now also U$9.P2-B, XBAT.2; no longer JP6.1, JP7.1
- net N$70: now also R22.1; no longer C203.2, DA2.2, DA2.4
- net T1: no longer DD6.1
- net T2: now also DD1.1, JP8.4; no longer DD1.2, DD6.2, JP8.2
- net T3: now also DD1.15, JP8.2; no longer DD1.1, DD6.3, JP8.3
- net T4: now also DD1.2, JP8.3; no longer DD1.15, DD6.4, JP8.4
Routing:
- net T3: track 0.00 -> 16.2 mm
- net N$16: track 0.00 -> 12.7 mm
- net T1: track 0.00 -> 8.75 mm
- net T4: track 0.00 -> 7.70 mm
- net T2: track 0.00 -> 7.67 mm
- net GND: track 34.1 -> 31.0 mm
- net N$5: track 13.0 -> 10.5 mm
- net VCC: track 49.1 -> 47.0 mm
- net N$121: track 17.0 -> 15.2 mm
- net N$8: track 16.4 -> 15.2 mm
- net N$7: track 3.81 -> 2.54 mm
- net N$6: track 3.81 -> 2.54 mm
- net +3V7: track 4.97 -> 3.91 mm
- net N$27: track 12.4 -> 11.6 mm
- net N$119: track 28.9 -> 28.3 mm
