File: K176IE13.brd (EAGLE design)
At the start: 95 parts, among them T1 TRAN_EE16, T3 TRAN_EE16

Commit message: .
Parts:
- removed T3: TRAN_EE16, ie13:EE16
- moved S2 12.7 mm to (-12.7, -18.4), turned to 180 degrees
- moved S3 12.7 mm to (12.7, -18.4)
- moved S4.1 12.7 mm to (-0.00, -18.4)
- moved S1 12.7 mm to (-25.4, -18.4), turned to 180 degrees
- moved D4 6.03 mm to (-21.6, -25.4), turned to 0 degrees
- moved R3 4.69 mm to (-16.8, -32.7)
- moved C3 4.27 mm to (-18.1, -30.5)
- moved R2 2.01 mm to (-29.2, -49.5)
- moved D3 1.91 mm to (-14.6, -29.2)
- moved R1 1.91 mm to (-21.6, -42.5)
- moved C11 1.42 mm to (-22.9, -42.5)
- moved C2 1.27 mm to (-29.2, -31.7)
- moved Z1 0.64 mm to (-29.2, -45.7)
Routing:
- net N$12: track 0.00 -> 46.5 mm, vias 0 -> 2
- net N$15: track 0.00 -> 21.1 mm
- net N$38: track 0.00 -> 15.5 mm
- net N$4: track 0.00 -> 8.40 mm
- net N$13: track 0.00 -> 8.40 mm
- net VCC: track 47.0 -> 55.4 mm
- net N$9: track 0.00 -> 8.40 mm
- net N$11: track 0.00 -> 8.40 mm
- net N$1: track 0.00 -> 7.28 mm
- net GND: track 31.0 -> 28.1 mm
Other:
- board outline added: 16.5 x 19 mm

Commit message: .
Parts:
- C5: value 10m -> (none)
Changed lines of the file:
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@@
 <element name="VT3" library="m_transistor" package="SOT23" value="BC847" x="13.968721875" y="-2.5387" rot="MR90"/>
 <element name="R7" library="rcl" package="M0805" value="270" x="13.9713" y="0.636278125" rot="MR180"/>
-<element name="C5" library="rcl" package="SANYO-OSCON_SMD_A5" value="10m" x="9.523721875" y="-1.2687" rot="MR270"/>
+<element name="C5" library="rcl" package="SANYO-OSCON_SMD_A5" value="" x="9.523721875" y="-1.2687" rot="MR270"/>
 <element name="JP1" library="Разъёмы штырьковые 2.54мм" package="1X07" value="" x="3.173721875" y="-10.7937" rot="R180"/>
 <element name="R8" library="rcl" package="M1206" value="0" x="12.063721875" y="3.8113" rot="MR270"/>

Commit message: .
Parts:
- added U$2: ULN2003C, DSS:DIL16_1
- added VT4: (no value), m_transistor:SOT23
- moved R8 37.0 mm to (-11.4, 32.4)
- moved R19 32.0 mm to (-26.7, 31.1)
- moved VT2 31.2 mm to (-18.4, 31.8)
- moved R3 16.1 mm to (-1.59, -37.8)
- moved XBAT 10.2 mm to (-6.35, 23.5)
- moved C3 2.54 mm to (-18.1, -27.9)
- moved D5 1.42 mm to (-1.90, 23.5), turned to 270 degrees
- moved C1 1.27 mm to (-29.2, -40.0)
- moved C2 0.71 mm to (-28.9, -32.4)
- moved R4 0.63 mm to (-1.91, -35.6)
- moved Z1 0.63 mm to (-29.2, -45.1)
Connections:
- removed net N$27: C5.+, R7.1, R8.2, VT1.2, VT3.2
- removed net N$70: R22.1
- removed net N$71: R23.1
- net +3V3: now also VT4.2
- net +3V7: now also VT4.3
- net GND: now also C5.+, R7.1, U$2.8, VT1.2, VT3.2
- net HE: now also R22.1
- net HK: now also R23.1
Routing:
- net +3V7: track 3.91 -> 25.9 mm
- net VCC: track 55.4 -> 74.0 mm
- net GND: track 28.1 -> 45.0 mm
- net N$27: track 11.6 -> 0.00 mm
- net N$3: track 0.00 -> 5.95 mm
- net N$2: track 0.00 -> 5.29 mm
- net N$119: track 28.3 -> 25.8 mm
- net N$121: track 15.2 -> 13.1 mm
- net N$1: track 7.28 -> 8.75 mm
- net T3: track 16.2 -> 16.8 mm

Commit message: .
Parts:
- added JP3, JP4: (no value), Разъёмы штырьковые 2.54мм:1X01
- moved U$2 76.6 mm to (-56.8, -22.2), turned to 270 degrees
- moved R8 42.9 mm to (8.89, -5.40), turned to 180 degrees
- moved C205 34.9 mm to (78.1, 16.5)
- moved R204 31.4 mm to (80.0, 22.2)
- moved R203 24.1 mm to (88.9, 23.5)
- moved D4 16.0 mm to (-5.72, -23.5), turned to 90 degrees
- moved VT4 13.4 mm to (-7.94, 0.64)
- moved R17 4.62 mm to (9.52, 30.5)
- moved R6 1.31 mm to (15.6, 1.91)
- moved VT1 1.27 mm to (14.0, -7.62)
- moved C5 1.14 mm to (10.2, -0.32)
- moved R7 1.00 mm to (14.3, -0.32)
- moved VT3 0.95 mm to (14.0, -3.49)
- moved DD4 0.90 mm to (1.25, -3.32)
- moved D5 0.63 mm to (-1.90, 24.1)
Connections:
- new net N$27: C5.+, R7.1, R8.2, VT1.2, VT3.2
- net A: now also DD4.16
- net B: now also DD4.15
- net C: now also DD4.14
- net D: now also DD4.13
- net E: now also DD4.12
- net F: now also DD4.11
- net G: now also DD4.10
- net GND: now also R8.1; no longer C5.+, R7.1, VT1.2, VT3.2
- net N$28: now also DD4.9; no longer R8.1, VT2.D
Routing:
- net B: track 58.4 -> 87.8 mm
- net A: track 68.7 -> 97.6 mm
- net C: track 61.0 -> 85.0 mm
- net G: track 63.5 -> 80.2 mm
- net F: track 65.2 -> 79.1 mm
- net +3V7: track 25.9 -> 38.7 mm
- net N$27: track 0.00 -> 12.0 mm
- net D: track 66.0 -> 75.3 mm
- net N$31: track 0.00 -> 8.12 mm
- net SD: track 0.00 -> 7.70 mm
- net N$32: track 0.00 -> 6.92 mm
- net N$68: track 0.00 -> 6.19 mm
- net N$33: track 0.00 -> 5.46 mm
- net N$26: track 0.00 -> 4.94 mm
- net N$67: track 0.00 -> 4.92 mm
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
Commit message: .
Parts:
- removed JP3, JP4: (no value), Разъёмы штырьковые 2.54мм:1X01
- removed R19: 100k, rcl:M0805
- removed VT2: (no value), m_transistor:DPACK
- added D10, D11: 1N4148DO35-7, diode:DO35-7
- moved U$9 6.36 mm to (-56.5, 4.13)
- moved U$2 5.02 mm to (-52.1, -23.8)
- moved VT4 1.93 mm to (-6.03, 0.32)
- renumbered JP1 to X2B, JP9 to X2A
Connections:
- new net HVCC: DD4.9, R6.1, T1.5, VT4.3
- new net N$70: D10.C, D11.C
- net +3V7: no longer R6.1, T1.5, VT4.3
- net GND: no longer R19.2, VT2.S
- net N$28: now also D11.A; no longer DD4.9
- net N$69: now also D10.A; no longer R19.1, VT2.G
Routing:
- net HVCC: track 0.00 -> 38.7 mm
- net +3V7: track 38.7 -> 0.00 mm

Commit message: .
Parts:
- added U$12, U$14, U$15, U$17, U$19, U$20, U$22, U$23, U$24, U$25, U$26, U$27, U$28, U$29, U$30, U$31, U$32, U$33, U$34, U$4, U$7: PAD, ie13:PAD-R
- added U$3, U$35: +, ie13:+
- moved D2 2.56 mm to (-10.5, -38.7)
- moved R21 1.27 mm to (3.81, 22.2)
- moved R23 0.95 mm to (0.95, 18.4)
- moved R22 0.71 mm to (2.86, 19.1)
- moved D1 0.71 mm to (-14.0, -37.8)
Connections:
- net H4 renamed H5
- new net A3: U$20.P$1, U$3.P$1, V3.6
- new net A5: U$28.P$1, V5.6
- new net B3: U$22.P$1, U$3.P$2, U$35.P$1, V3.5
- new net B5: U$29.P$1, V5.5
- new net C3: U$23.P$1, V3.4
- new net C5: U$30.P$1, V5.4
- new net D3: U$24.P$1, V3.2
- new net D5: U$31.P$1, V5.2
- new net E3: U$25.P$1, V3.1
- new net E5: U$32.P$1, V5.1
- new net F3: U$26.P$1, V3.10
- new net F5: U$33.P$1, V5.10
- new net G3: U$27.P$1, U$35.P$2, V3.3
- new net G5: U$34.P$1, V5.3
- net A: now also U$4.P$1; no longer V5.6
- net B: now also U$7.P$1; no longer V5.5
- net C: now also U$12.P$1; no longer V5.4
- net D: now also U$14.P$1; no longer V5.2
- net E: now also U$15.P$1; no longer V5.1
- net F: now also U$17.P$1; no longer V5.10
- net G: now also U$19.P$1; no longer V5.3
- net H3: now also V3.11
Routing:
- net B: track 87.8 -> 58.1 mm, vias 4 -> 2
- net C: track 85.0 -> 55.8 mm, vias 4 -> 2
- net G: track 80.2 -> 51.6 mm, vias 4 -> 2
- net D: track 75.3 -> 47.4 mm, vias 4 -> 2
- net E: track 72.3 -> 45.0 mm, vias 4 -> 2
- net B3: track 0.00 -> 12.0 mm
- net G3: track 0.00 -> 4.46 mm
- net B5: track 0.00 -> 4.45 mm
- net A: track 97.6 -> 93.1 mm
- net A5: track 0.00 -> 4.44 mm
- net D3: track 0.00 -> 4.07 mm
- net A3: track 0.00 -> 3.96 mm
- net C3: track 0.00 -> 3.88 mm
- net C5: track 0.00 -> 3.81 mm
- net F: track 79.1 -> 75.5 mm
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
Commit message: .
Parts:
- added U$36, U$37, U$38, U$39, U$40, U$41, U$42, U$43, U$44, U$45, U$46, U$47, U$48, U$49: PAD, ie13:PAD-R
- moved U$2 6.43 mm to (-58.1, -21.6)
- renumbered JP2 to X1B, JP8 to X1A
Connections:
- removed net A: DD4.16, U$4.P$1, V1.6, V2.6, V4.6
- removed net B: DD4.15, U$7.P$1, V1.5, V2.5, V4.5
- removed net C: DD4.14, U$12.P$1, V1.4, V2.4, V4.4
- removed net D: DD4.13, U$14.P$1, V1.2, V2.2, V4.2
- removed net E: DD4.12, U$15.P$1, V1.1, V2.1, V4.1
- removed net F: DD4.11, U$17.P$1, V1.10, V2.10, V4.10
- removed net G: DD4.10, U$19.P$1, V1.3, V2.3, V4.3
- new net A1: U$4.P$1, V1.6
- new net A2: U$36.P$1, V2.6
- new net A4: DD4.16, U$43.P$1, V4.6
- new net B1: U$7.P$1, V1.5
- new net B2: U$37.P$1, V2.5
- new net B4: DD4.15, U$44.P$1, V4.5
- new net C1: U$12.P$1, V1.4
- new net C2: U$38.P$1, V2.4
- new net C4: DD4.14, U$45.P$1, V4.4
- new net D1: U$14.P$1, V1.2
- new net D2: U$39.P$1, V2.2
- new net D4: DD4.13, U$46.P$1, V4.2
- new net E1: U$15.P$1, V1.1
- new net E2: U$40.P$1, V2.1
- new net E4: DD4.12, U$47.P$1, V4.1
- new net F1: U$17.P$1, V1.10
- new net F2: U$41.P$1, V2.10
- new net F4: DD4.11, U$48.P$1, V4.10
- new net G1: U$19.P$1, V1.3
- new net G2: U$42.P$1, V2.3
- new net G4: DD4.10, U$49.P$1, V4.3
- new net H4: V4.11
- net B3: now also DD6.15
- net D3: now also DD6.16
- net H3: no longer V4.11
Routing:
- net A: track 93.1 -> 0.00 mm, vias 4 -> 0
- net F: track 75.5 -> 0.00 mm, vias 4 -> 0
- net A4: track 0.00 -> 70.5 mm, vias 0 -> 3
- net F4: track 0.00 -> 60.4 mm, vias 0 -> 3
- net B: track 58.1 -> 0.00 mm, vias 2 -> 0
- net C: track 55.8 -> 0.00 mm, vias 2 -> 0
- net G: track 51.6 -> 0.00 mm, vias 2 -> 0
- net D: track 47.4 -> 0.00 mm, vias 2 -> 0
- net E: track 45.0 -> 0.00 mm, vias 2 -> 0
- net B4: track 0.00 -> 23.6 mm
- net C4: track 0.00 -> 21.6 mm
- net G4: track 0.00 -> 19.9 mm
- net D4: track 0.00 -> 16.9 mm
- net E4: track 0.00 -> 14.4 mm
- net B2: track 0.00 -> 4.63 mm
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
Commit message: .
Parts:
- added U$50: +, ie13:+
- added U$51, U$52, U$53, U$54, U$55: PAD, ie13:PAD-R
- moved DD50 28.3 mm to (60.0, 2.22)
- moved U$3 10.9 mm to (-5.40, 9.21)
- moved U$9 7.73 mm to (-64.1, 5.40)
- moved U$35 1.00 mm to (-0.32, 8.89)
- moved VT4 0.95 mm to (-6.03, 1.27)
- moved U$45 0.32 mm to (15.2, 8.89)
Connections:
- net N$72 renamed T1B
- net N$73 renamed T3B
- net N$74 renamed T4B
- net N$75 renamed T2B
- new net HE1: U$51.P$1, V1.7
- new net HE2: U$53.P$1, V2.7
- new net HK1: U$52.P$1, V1.8
- new net HK2: U$54.P$1, V2.8
- net A3: now also DD6.15, U$55.P$1; no longer U$3.P$1
- net B3: no longer DD6.15, U$3.P$2, U$35.P$1
- net C3: now also U$35.P$1
- net D3: now also U$3.P$1, U$50.P$2
- net E3: now also U$3.P$2
- net G2: now also DD4.10
- net G3: now also U$50.P$1
- net G4: no longer DD4.10
- net HE: no longer V1.7, V2.7
- net HK: no longer V1.8, V2.8
Routing:
- net F4: track 60.4 -> 35.0 mm, vias 3 -> 2
- net HE: track 68.4 -> 47.4 mm, vias 5 -> 4
- net HK: track 66.5 -> 46.7 mm, vias 5 -> 4
- net G4: track 19.9 -> 3.17 mm
- net D3: track 4.07 -> 19.3 mm, vias 0 -> 1
- net G2: track 3.17 -> 17.7 mm
- net B3: track 12.0 -> 2.56 mm
- net HE1: track 0.00 -> 3.81 mm
- net F2: track 0.00 -> 3.59 mm
- net HK1: track 0.00 -> 3.17 mm
- net E3: track 2.01 -> 3.63 mm
- net C3: track 3.88 -> 5.50 mm
- net G3: track 4.46 -> 6.03 mm
- net A3: track 3.96 -> 2.54 mm
- net E4: track 14.4 -> 15.8 mm
