File: K176IE13.brd (EAGLE design)
At the start: 16.5 x 19 mm, 139 parts, among them T1 TRAN_EE16

Commit message: .
Parts:
- moved U$9 3.42 mm to (-62.9, 8.57)
- moved VT4 0.32 mm to (-5.71, 1.27)
- renumbered R8 to J2
Routing:
- net HVCC: track 38.7 -> 46.0 mm
- net A4: track 70.5 -> 73.4 mm, vias 3 -> 2
Changed lines of the file:
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@@
 <wire x1="-25.4" y1="18.415" x2="-12.065" y2="18.415" width="0.254" layer="51"/>
 <wire x1="-22.86" y1="19.05" x2="-9.525" y2="19.05" width="0.254" layer="51"/>
+<wire x1="3.81" y1="10.4775" x2="3.81" y2="13.97" width="0.254" layer="51"/>
+<wire x1="3.81" y1="13.97" x2="-3.81" y2="13.97" width="0.254" layer="51"/>
+<wire x1="-3.81" y1="13.97" x2="-3.81" y2="16.51" width="0.254" layer="51"/>
+<wire x1="-3.81" y1="16.51" x2="-2.54" y2="17.78" width="0.254" layer="51"/>
 </plain>
 <attributes>
@@
 <element name="C5" library="rcl" package="SANYO-OSCON_SMD_A5" value="" x="10.158721875" y="-0.3162" rot="MR270"/>
 <element name="X2B" library="Разъёмы штырьковые 2.54мм" package="1X07" value="" x="3.173721875" y="-10.7937" rot="R180"/>
-<element name="R8" library="rcl" package="M1206" value="0" x="8.8887" y="-5.398778125" rot="MR180"/>
+<element name="J2" library="rcl" package="M1206" value="0" x="8.8887" y="-5.398778125" rot="MR180"/>
 <element name="U$13" library="MT3608" package="SOT23-6" value="MT3608SOT23-6" x="13.968721875" y="23.4963" rot="MR0"/>
 <element name="L1" library="rcl" package="L3225M" value="" x="17.778721875" y="23.4963" rot="MR270"/>
@@
 <element name="R20" library="rcl" package="M0805" value="2k2" x="8.888721875" y="25.4013" rot="MR90"/>
 <element name="C14" library="rcl" package="C1206" value="" x="6.3487" y="22.858721875" rot="MR180"/>
-<element name="U$9" library="TP4056+mod" package="MOD_03962A" value="MOD_TP4056" x="-64.136278125" y="5.3988" rot="MR270"/>
+<element name="U$9" library="TP4056+mod" package="MOD_03962A" value="MOD_TP4056" x="-62.866278125" y="8.5738" rot="MR270"/>
 <element name="R21" library="rcl" package="M0805" value="" x="3.808721875" y="22.2263" rot="MR0"/>
 <element name="S3" library="switch" package="SKHMPXE010" value="УЧ" x="12.698721875" y="-18.4137" rot="MR0"/>
@@
 <element name="X1B" library="Разъёмы штырьковые 2.54мм" package="1X04" value="" x="-10.16" y="-6.985" rot="R270"/>
 <element name="U$2" library="DSS" package="DIL16_1" value="ULN2003C" x="-58.1025" y="-21.59" rot="R270"/>
-<element name="VT4" library="m_transistor" package="SOT23" value="" x="-6.0325" y="1.27" rot="MR90"/>
+<element name="VT4" library="m_transistor" package="SOT23" value="" x="-5.715" y="1.27" rot="MR90"/>
 <element name="D10" library="diode" package="DO35-7" value="1N4148DO35-7" x="-60.0075" y="-41.275"/>
 <element name="D11" library="diode" package="DO35-7" value="1N4148DO35-7" x="-61.2775" y="-45.72"/>
@@
 <contactref element="U$2" pad="8"/>
 <contactref element="DD4" pad="8"/>
-<contactref element="R8" pad="1"/>
+<contactref element="J2" pad="1"/>
 <wire x1="7.4887" y1="-5.398778125" x2="5.899921875" y2="-3.81" width="0.4064" layer="16"/>
 <wire x1="5.899921875" y1="-3.81" x2="-3.191278125" y2="-3.81" width="0.4064" layer="16"/>
@@
 <wire x1="14.736278125" y1="26.0337" x2="13.968721875" y2="22.4963" width="0" layer="19" extent="16-16"/>
 <wire x1="-61.9125" y1="-30.48" x2="-29.211278125" y2="-39.0537" width="0" layer="19" extent="16-16"/>
-<wire x1="-46.016278125" y1="10.8988" x2="-14.072878125" y2="-11.4287" width="0" layer="19" extent="16-16"/>
+<wire x1="-44.746278125" y1="14.0738" x2="-14.072878125" y2="-11.4287" width="0" layer="19" extent="16-16"/>
 </signal>
 <signal name="VCC">
@@
 <contactref element="U$9" pad="P2+OUT"/>
 <contactref element="VT4" pad="2"/>
-<wire x1="-7.1325" y1="2.22" x2="-46.016278125" y2="-0.1012" width="0" layer="19" extent="16-16"/>
-<wire x1="11.468721875" y1="21.4963" x2="-7.1325" y2="2.22" width="0" layer="19" extent="16-16"/>
+<wire x1="-6.815" y1="2.22" x2="-44.746278125" y2="3.0738" width="0" layer="19" extent="16-16"/>
+<wire x1="11.468721875" y1="21.4963" x2="-6.815" y2="2.22" width="0" layer="19" extent="16-16"/>
 <wire x1="11.468721875" y1="22.4963" x2="11.468721875" y2="21.4963" width="0" layer="19" extent="16-16"/>
 <wire x1="11.936278125" y1="26.0337" x2="11.468721875" y2="22.4963" width="0" layer="19" extent="16-16"/>
@@
 <contactref element="U$9" pad="P2+B"/>
 <contactref element="XBAT" pad="1"/>
-<wire x1="-6.35" y1="22.225" x2="-46.016278125" y2="2.8988" width="0" layer="19" extent="1-1"/>
+<wire x1="-6.35" y1="22.225" x2="-44.746278125" y2="6.0738" width="0" layer="19" extent="1-1"/>
 </signal>
 <signal name="N$47">
 <contactref element="XBAT" pad="2"/>
 <contactref element="U$9" pad="P2-B"/>
-<wire x1="-6.35" y1="24.765" x2="-46.016278125" y2="7.8988" width="0" layer="19" extent="1-1"/>
+<wire x1="-6.35" y1="24.765" x2="-44.746278125" y2="11.0738" width="0" layer="19" extent="1-1"/>
 </signal>
 <signal name="T1B">
@@
 <contactref element="R7" pad="1"/>
 <contactref element="C5" pad="+"/>
-<contactref element="R8" pad="2"/>
+<contactref element="J2" pad="2"/>
 <wire x1="12.868721875" y1="-2.5412" x2="12.868721875" y2="-1.5837" width="0.4064" layer="16"/>
 <wire x1="10.158721875" y1="-2.1162" x2="10.158721875" y2="-2.8575" width="0.4064" layer="16"/>
@@
 <wire x1="6.985" y1="2.8575" x2="6.985" y2="-1.5875" width="0.4064" layer="16"/>
 <wire x1="6.985" y1="-1.5875" x2="6.0325" y2="-2.54" width="0.4064" layer="16"/>
-<wire x1="6.0325" y1="-2.54" x2="-3.4925" y2="-2.54" width="0.4064" layer="16"/>
+<wire x1="6.0325" y1="-2.54" x2="-3.191278125" y2="-2.54" width="0.4064" layer="16"/>
 <wire x1="6.985" y1="2.8575" x2="8.89" y2="4.7625" width="0.4064" layer="16"/>
 <wire x1="8.89" y1="4.7625" x2="17.145" y2="4.7625" width="0.4064" layer="16"/>
@@
 <wire x1="17.4625" y1="5.08" x2="20.32" y2="5.08" width="0.4064" layer="16"/>
 <contactref element="DD4" pad="9"/>
-<wire x1="-3.191278125" y1="-0.2428" x2="-4.9325" y2="1.27" width="0" layer="19" extent="16-16"/>
-<wire x1="-3.4925" y1="-2.54" x2="-3.191278125" y2="-0.2428" width="0" layer="19" extent="16-16"/>
+<wire x1="-3.191278125" y1="-2.54" x2="-3.191278125" y2="-0.2428" width="0.4064" layer="16"/>
+<wire x1="-4.615" y1="1.27" x2="-4.615" y2="-2.54" width="0.4064" layer="16"/>
+<wire x1="-4.615" y1="-2.54" x2="-3.191278125" y2="-2.54" width="0.4064" layer="16"/>
 </signal>
 <signal name="N$28">
@@
 <contactref element="V4" pad="6"/>
 <via x="-6.986278125" y="19.6863" extent="1-16" drill="0.6" diameter="2.1844"/>
-<via x="30.478721875" y="19.6863" extent="1-16" drill="0.6" diameter="2.1844"/>
-<wire x1="30.478721875" y1="19.6863" x2="19.048721875" y2="19.6863" width="0.4064" layer="1"/>
 <via x="19.048721875" y="19.6863" extent="1-16" drill="0.6" diameter="2.1844"/>
 <wire x1="-6.986278125" y1="19.6863" x2="19.048721875" y2="19.6863" width="0.4064" layer="1"/>
@@
 <wire x1="17.78" y1="15.24" x2="19.05" y2="13.97" width="0.4064" layer="16"/>
 <contactref element="U$43" pad="P$1"/>
-<wire x1="30.478721875" y1="19.6863" x2="30.48" y2="19.685" width="0" layer="19" extent="16-16"/>
+<wire x1="30.48" y1="19.685" x2="26.9875" y2="23.1775" width="0.4064" layer="16"/>
+<wire x1="26.9875" y1="23.1775" x2="23.8125" y2="23.1775" width="0.4064" layer="16"/>
+<wire x1="23.8125" y1="23.1775" x2="20.32" y2="19.685" width="0.4064" layer="16"/>
+<wire x1="20.32" y1="19.685" x2="19.050021875" y2="19.685" width="0.4064" layer="16"/>
+<wire x1="19.050021875" y1="19.685" x2="19.048721875" y2="19.6863" width="0.4064" layer="16"/>
 </signal>
 <signal name="B4">

Commit message: .
Parts:
- removed U$13: MT3608SOT23-6, MT3608:SOT23-6
- added DA1: MT3608SOT23-6, MT3608:SOT23-6
- added U$56, U$57, U$58, U$59, U$60, U$61, U$62, U$63, U$64, U$65, U$66: PAD, ie13:PAD-R
- added U$67: +, ie13:+
- moved U$43 12.7 mm to (17.8, 19.7)
- moved U$48 12.7 mm to (10.2, 17.8)
- moved VT4 1.42 mm to (-5.08, 2.54)
- moved L1 1.42 mm to (19.0, 24.1)
- moved C6 0.89 mm to (14.0, 25.4), turned to 0 degrees
Connections:
- new net HE4: U$64.P$1, V4.7
- new net HE5: U$57.P$1, V5.7
- new net HK4: U$66.P$1, V4.8
- new net HK5: U$56.P$1, V5.8
- net +3V3: now also DA1.4, DA1.5; no longer U$13.4, U$13.5
- net A4: now also U$67.P$1
- net A5: now also U$67.P$2
- net GND: now also DA1.2; no longer U$13.2
- net HE: no longer V4.7, V5.7
- net HK: no longer V4.8, V5.8
- net N$34: now also DA1.1; no longer U$13.1
- net N$44: now also DA1.3; no longer U$13.3
Routing:
- net HE: track 47.4 -> 0.00 mm, vias 4 -> 0
- net HK: track 46.7 -> 0.00 mm, vias 4 -> 0
- net A4: track 73.4 -> 41.5 mm, vias 2 -> 0
- net F4: track 35.0 -> 22.3 mm, vias 2 -> 0
- net D3: track 19.3 -> 27.9 mm, vias 1 -> 2
- net A5: track 4.44 -> 9.10 mm
- net A2: track 0.00 -> 4.49 mm
- net HE2: track 0.00 -> 3.86 mm
- net HE4: track 0.00 -> 3.81 mm
- net HE5: track 0.00 -> 3.81 mm
- net HK2: track 0.00 -> 3.24 mm
- net HK4: track 0.00 -> 3.17 mm
- net HK5: track 0.00 -> 3.17 mm
- net HVCC: track 46.0 -> 44.3 mm
- net G2: track 17.7 -> 19.1 mm

Commit message: .
Parts:
- added J3: 0, rcl:M1206
- added U$13, U$68, U$69, U$70: PAD, ie13:PAD-R
- R17: device rcl:RTRIM3296W -> rcl:RTRIM3296P
- moved U$6 40.9 mm to (80.6, -1.27), turned to 90 degrees
- moved C10 39.7 mm to (57.8, -60.3)
- moved D6 39.7 mm to (76.8, -69.2)
- moved D7 39.7 mm to (61.0, -74.9)
- moved D8 39.7 mm to (61.6, -67.3)
- moved D9 39.7 mm to (68.6, -53.3)
- moved R10 39.7 mm to (70.5, -58.4)
- moved R11 39.7 mm to (74.3, -65.4)
- moved R12 39.7 mm to (74.3, -74.9)
- moved R14 39.7 mm to (67.3, -76.2)
- moved R15 39.7 mm to (73.7, -51.4)
- moved R9 39.7 mm to (57.1, -78.1)
- moved C7 39.7 mm to (80.6, -64.8)
- moved C8 39.7 mm to (68.6, -79.4)
- moved C9 39.7 mm to (76.2, -57.8)
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Connections:
- net B4: now also J3.1
- net B5: now also J3.2
- net S1: now also U$13.P$1
- net S2: now also U$68.P$1
- net S3: now also U$69.P$1
- net S4: now also U$70.P$1
Routing:
- net A4: track 41.5 -> 48.9 mm
- net B5: track 4.45 -> 10.7 mm
- net B4: track 23.6 -> 28.6 mm
- net D3: track 27.9 -> 24.1 mm
- net A5: track 9.10 -> 12.4 mm
- net S3: track 0.00 -> 2.71 mm
- net S2: track 0.00 -> 2.71 mm
- net S1: track 0.00 -> 2.71 mm
- net S4: track 0.00 -> 2.42 mm
- net T2: track 7.67 -> 5.80 mm
- net T4: track 7.70 -> 5.98 mm
- net T3: track 16.8 -> 15.0 mm
- net T1: track 8.75 -> 7.03 mm
- net F2: track 3.59 -> 5.04 mm
- net F1: track 3.59 -> 5.04 mm
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
Commit message: .
Parts:
- removed U$58: PAD, ie13:PAD-R
- moved U$59 52.1 mm to (-25.4, -10.2)
- moved U$60 47.7 mm to (-27.9, -8.89)
- moved U$61 44.9 mm to (-25.4, -7.62)
- moved U$62 40.5 mm to (-27.9, -6.35)
- moved U$55 1.27 mm to (-25.4, -5.08)
- moved D2 0.90 mm to (-9.84, -38.1)
Connections:
- net A3: now also DD6.14; no longer DD6.15
- net D3: now also DD6.15; no longer DD6.16
- net S1: now also DD6.11, U$60.P$1
- net S2: now also DD6.12, U$61.P$1
- net S3: now also DD6.10, U$59.P$1
- net S4: now also DD6.13, U$62.P$1

Commit message: .
Parts:
- moved X1A 1.31 mm to (-11.7, -48.3)
- moved X1B 0.95 mm to (-12.1, -6.03)
- moved U$9 0.64 mm to (-26.4, -3.49)
Routing:
- net GND: track 49.4 -> 66.2 mm
Changed lines of the file:
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@@
 <element name="C205" library="rcl" package="E2,5-5" value="100m" x="78.103721875" y="16.5113"/>
 <element name="C201" library="rcl" package="E3,5-8" value="470m" x="102.233721875" y="22.8613"/>
-<element name="X1A" library="Разъёмы штырьковые 2.54мм" package="1X04" value="" x="-12.063721875" y="-49.5313" rot="R270"/>
+<element name="X1A" library="Разъёмы штырьковые 2.54мм" package="1X04" value="" x="-11.746221875" y="-48.2613" rot="R270"/>
 <element name="X2A" library="Разъёмы штырьковые 2.54мм" package="1X07" value="" x="3.173721875" y="-53.3387"/>
 <element name="DD40" library="40xx" package="SO14" value="4011D" x="57.148721875" y="-47.6237" rot="MR180"/>
@@
 <element name="R20" library="rcl" package="M0805" value="2k2" x="6.348721875" y="32.7038" rot="MR90"/>
 <element name="C14" library="rcl" package="C1206" value="" x="5.0787" y="30.161221875" rot="MR180"/>
-<element name="U$9" library="TP4056+mod" package="MOD_03962A" value="MOD_TP4056" x="-25.718778125" y="-3.4912" rot="MR270"/>
+<element name="U$9" library="TP4056+mod" package="MOD_03962A" value="MOD_TP4056" x="-26.353778125" y="-3.4912" rot="MR270"/>
 <element name="R21" library="rcl" package="M0805" value="" x="3.491221875" y="22.2263" rot="MR0"/>
 <element name="S3" library="switch" package="SKHMPXE010" value="УЧ" x="12.698721875" y="-18.4137" rot="MR0"/>
@@
 <element name="R22" library="rcl" package="M0805" value="" x="2.8575" y="19.05" rot="MR270"/>
 <element name="R23" library="rcl" package="M0805" value="" x="0.9525" y="18.415" rot="MR270"/>
-<element name="X1B" library="Разъёмы штырьковые 2.54мм" package="1X04" value="" x="-12.065" y="-6.985" rot="R270"/>
+<element name="X1B" library="Разъёмы штырьковые 2.54мм" package="1X04" value="" x="-12.065" y="-6.0325" rot="R270"/>
 <element name="U$2" library="DSS" package="DIL16_1" value="ULN2003C" x="-58.1025" y="-21.59" rot="R270"/>
 <element name="VT4" library="m_transistor" package="SOT23" value="" x="-5.08" y="2.54" rot="MR90"/>
@@
 <wire x1="6.348721875" y1="31.7538" x2="6.4787" y2="30.161221875" width="0" layer="19" extent="16-16"/>
 <wire x1="5.899921875" y1="-3.81" x2="15.876278125" y2="25.4462" width="0" layer="19" extent="16-16"/>
-<wire x1="-7.598778125" y1="2.0088" x2="-3.191278125" y2="-3.81" width="0" layer="19" extent="16-16"/>
-<wire x1="-16.612878125" y1="-11.4287" x2="-3.191278125" y2="-6.3896" width="0" layer="19" extent="16-16"/>
+<wire x1="-8.233778125" y1="2.0088" x2="-3.191278125" y2="-3.81" width="0" layer="19" extent="16-16"/>
 <wire x1="-19.048778125" y1="-27.9387" x2="-16.612878125" y2="-11.4287" width="0" layer="19" extent="16-16"/>
 <wire x1="-17.781278125" y1="-34.9237" x2="-19.048778125" y2="-27.9387" width="0" layer="19" extent="16-16"/>
@@
 <wire x1="5.7137" y1="-37.146278125" x2="-2.538778125" y2="-37.7812" width="0" layer="19" extent="16-16"/>
 <wire x1="-61.9125" y1="-30.48" x2="-29.211278125" y2="-39.0537" width="0" layer="19" extent="16-16"/>
+<wire x1="-3.191278125" y1="-6.3896" x2="-3.5321" y2="-6.3896" width="0.4064" layer="16"/>
+<wire x1="-3.5321" y1="-6.3896" x2="-6.35" y2="-9.2075" width="0.4064" layer="16"/>
+<wire x1="-6.35" y1="-9.2075" x2="-6.35" y2="-11.1125" width="0.4064" layer="16"/>
+<wire x1="-6.35" y1="-11.1125" x2="-6.985" y2="-11.7475" width="0.4064" layer="16"/>
+<wire x1="-6.985" y1="-11.7475" x2="-14.2875" y2="-11.7475" width="0.4064" layer="16"/>
+<wire x1="-14.2875" y1="-11.7475" x2="-15.24" y2="-11.43" width="0.4064" layer="16"/>
+<wire x1="-15.24" y1="-11.43" x2="-16.611578125" y2="-11.43" width="0.4064" layer="16"/>
+<wire x1="-16.611578125" y1="-11.43" x2="-16.612878125" y2="-11.4287" width="0.4064" layer="16"/>
 </signal>
 <signal name="VCC">
@@
 <contactref element="DD1" pad="3"/>
 <contactref element="X1A" pad="1"/>
-<wire x1="-12.7" y1="-45.085" x2="-12.063721875" y2="-45.7213" width="0.4064" layer="16"/>
+<wire x1="-12.7" y1="-45.085" x2="-11.746221875" y2="-44.4513" width="0.4064" layer="16"/>
 <wire x1="-17.781278125" y1="-47.6237" x2="-17.1437" y2="-47.6237" width="0.4064" layer="16"/>
 <wire x1="-17.1437" y1="-47.6237" x2="-14.605" y2="-45.085" width="0.4064" layer="16"/>
@@
 <contactref element="DD1" pad="15"/>
 <contactref element="X1A" pad="2"/>
-<wire x1="-12.063721875" y1="-48.2613" x2="-12.6987" y2="-47.6263" width="0.4064" layer="16"/>
+<wire x1="-11.746221875" y1="-46.9913" x2="-12.6987" y2="-47.6263" width="0.4064" layer="16"/>
 <wire x1="-12.6987" y1="-47.6263" x2="-13.97" y2="-47.625" width="0.4064" layer="16"/>
 <wire x1="-13.97" y1="-47.625" x2="-15.875" y2="-48.895" width="0.4064" layer="16"/>
@@
 <contactref element="DD1" pad="1"/>
 <contactref element="X1A" pad="4"/>
-<wire x1="-12.063721875" y1="-53.3413" x2="-14.601121875" y2="-52.7037" width="0.4064" layer="16"/>
+<wire x1="-11.746221875" y1="-52.0713" x2="-14.601121875" y2="-52.7037" width="0.4064" layer="16"/>
 <wire x1="-14.601121875" y1="-52.7037" x2="-17.781278125" y2="-52.7037" width="0.4064" layer="16"/>
-<wire x1="-9.843778125" y1="-39.7987" x2="-12.063721875" y2="-53.3413" width="0" layer="19" extent="16-16"/>
+<wire x1="-9.843778125" y1="-39.7987" x2="-11.746221875" y2="-52.0713" width="0" layer="19" extent="16-16"/>
 </signal>
 <signal name="N$9">
@@
 <contactref element="DD1" pad="2"/>
 <contactref element="X1A" pad="3"/>
-<wire x1="-12.063721875" y1="-50.8013" x2="-12.7013" y2="-50.1663" width="0.4064" layer="16"/>
+<wire x1="-11.746221875" y1="-49.5313" x2="-12.7013" y2="-50.1663" width="0.4064" layer="16"/>
 <wire x1="-12.7013" y1="-50.1663" x2="-12.7" y2="-50.165" width="0.4064" layer="16"/>
 <wire x1="-12.7" y1="-50.165" x2="-17.779978125" y2="-50.165" width="0.4064" layer="16"/>
@@
 <wire x1="22.5438" y1="23.683778125" x2="18.5437" y2="22.541221875" width="0" layer="19" extent="16-16"/>
 <wire x1="-6.18" y1="3.49" x2="18.5437" y2="22.541221875" width="0" layer="19" extent="16-16"/>
-<wire x1="-7.598778125" y1="-8.9912" x2="-6.18" y2="3.49" width="0" layer="19" extent="16-16"/>
+<wire x1="-8.233778125" y1="-8.9912" x2="-6.18" y2="3.49" width="0" layer="19" extent="16-16"/>
 </signal>
 <signal name="SD">
@@
 <contactref element="U$9" pad="P2+B"/>
 <contactref element="XBAT" pad="1"/>
-<wire x1="-7.598778125" y1="-5.9912" x2="-8.89" y2="23.1775" width="0" layer="19" extent="1-1"/>
+<wire x1="-8.233778125" y1="-5.9912" x2="-8.89" y2="23.1775" width="0" layer="19" extent="1-1"/>
 </signal>
 <signal name="N$47">
 <contactref element="XBAT" pad="2"/>
 <contactref element="U$9" pad="P2-B"/>
-<wire x1="-7.598778125" y1="-0.9912" x2="-8.89" y2="25.7175" width="0" layer="19" extent="1-1"/>
+<wire x1="-8.233778125" y1="-0.9912" x2="-8.89" y2="25.7175" width="0" layer="19" extent="1-1"/>
 </signal>
 <signal name="T1B">
 <contactref element="DD6" pad="4"/>
 <contactref element="X1B" pad="1"/>
-<wire x1="-12.065" y1="-3.175" x2="-16.612878125" y2="-6.3487" width="0" layer="19" extent="16-16"/>
+<wire x1="-12.065" y1="-2.2225" x2="-16.612878125" y2="-6.3487" width="0" layer="19" extent="16-16"/>
 </signal>
 <signal name="T3B">
 <contactref element="DD6" pad="5"/>
 <contactref element="X1B" pad="2"/>
-<wire x1="-12.065" y1="-5.715" x2="-16.612878125" y2="-7.6187" width="0" layer="19" extent="16-16"/>
+<wire x1="-12.065" y1="-4.7625" x2="-16.612878125" y2="-7.6187" width="0" layer="19" extent="16-16"/>
 </signal>
 <signal name="T4B">
 <contactref element="DD6" pad="6"/>
 <contactref element="X1B" pad="3"/>
-<wire x1="-12.065" y1="-8.255" x2="-16.612878125" y2="-8.8887" width="0" layer="19" extent="16-16"/>
+<wire x1="-12.065" y1="-7.3025" x2="-16.612878125" y2="-8.8887" width="0" layer="19" extent="16-16"/>
 </signal>
 <signal name="T2B">
 <contactref element="DD6" pad="7"/>
 <contactref element="X1B" pad="4"/>
-<wire x1="-12.065" y1="-10.795" x2="-16.612878125" y2="-10.1587" width="0" layer="19" extent="16-16"/>
+<wire x1="-12.065" y1="-9.8425" x2="-16.612878125" y2="-10.1587" width="0" layer="19" extent="16-16"/>
 </signal>
 <signal name="N$27">
