File: K176IE13.brd (EAGLE design)
At the start: 16.5 x 19 mm, 155 parts, among them J2 0, J3 0, T1 TRAN_EE16

Commit message: .
Parts:
- added U$58: PAD, ie13:PAD-R
- moved VT4 0.32 mm to (-4.76, 2.54)
Connections:
- net HVCC: now also DD6.9, U$58.P$1
Routing:
- net HVCC: track 43.9 -> 45.3 mm
Changed lines of the file:
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@@
 <element name="X1B" library="Разъёмы штырьковые 2.54мм" package="1X04" value="" x="-12.065" y="-6.0325" rot="R270"/>
 <element name="U$2" library="DSS" package="DIL16_1" value="ULN2003C" x="-58.1025" y="-21.59" rot="R270"/>
-<element name="VT4" library="m_transistor" package="SOT23" value="" x="-5.08" y="2.54" rot="MR90"/>
+<element name="VT4" library="m_transistor" package="SOT23" value="" x="-4.7625" y="2.54" rot="MR90"/>
 <element name="D10" library="diode" package="DO35-7" value="1N4148DO35-7" x="-60.0075" y="-41.275"/>
 <element name="D11" library="diode" package="DO35-7" value="1N4148DO35-7" x="-61.2775" y="-45.72"/>
@@
 <element name="U$69" library="ie13" package="PAD-R" value="PAD" x="11.1125" y="17.78" rot="R90"/>
 <element name="U$70" library="ie13" package="PAD-R" value="PAD" x="23.8125" y="17.4625" rot="R90"/>
+<element name="U$58" library="ie13" package="PAD-R" value="PAD" x="-4.7625" y="-0.3175"/>
 </elements>
 <signals>
@@
 <wire x1="-3.191278125" y1="-3.81" x2="-3.191278125" y2="-6.3896" width="0.4064" layer="16"/>
 <contactref element="DD6" pad="8"/>
+<wire x1="-3.191278125" y1="-6.3896" x2="-3.5321" y2="-6.3896" width="0.4064" layer="16"/>
+<wire x1="-3.5321" y1="-6.3896" x2="-6.35" y2="-9.2075" width="0.4064" layer="16"/>
+<wire x1="-6.35" y1="-9.2075" x2="-6.35" y2="-11.1125" width="0.4064" layer="16"/>
+<wire x1="-6.35" y1="-11.1125" x2="-6.985" y2="-11.7475" width="0.4064" layer="16"/>
+<wire x1="-6.985" y1="-11.7475" x2="-14.2875" y2="-11.7475" width="0.4064" layer="16"/>
+<wire x1="-14.2875" y1="-11.7475" x2="-15.24" y2="-11.43" width="0.4064" layer="16"/>
+<wire x1="-15.24" y1="-11.43" x2="-16.611578125" y2="-11.43" width="0.4064" layer="16"/>
+<wire x1="-16.611578125" y1="-11.43" x2="-16.612878125" y2="-11.4287" width="0.4064" layer="16"/>
 <wire x1="95.248721875" y1="12.6413" x2="104.011721875" y2="22.8613" width="0" layer="19" extent="16-16"/>
 <wire x1="92.708721875" y1="12.6413" x2="95.248721875" y2="12.6413" width="0" layer="19" extent="16-16"/>
@@
 <wire x1="5.7137" y1="-37.146278125" x2="-2.538778125" y2="-37.7812" width="0" layer="19" extent="16-16"/>
 <wire x1="-61.9125" y1="-30.48" x2="-29.211278125" y2="-39.0537" width="0" layer="19" extent="16-16"/>
-<wire x1="-3.191278125" y1="-6.3896" x2="-3.5321" y2="-6.3896" width="0.4064" layer="16"/>
-<wire x1="-3.5321" y1="-6.3896" x2="-6.35" y2="-9.2075" width="0.4064" layer="16"/>
-<wire x1="-6.35" y1="-9.2075" x2="-6.35" y2="-11.1125" width="0.4064" layer="16"/>
-<wire x1="-6.35" y1="-11.1125" x2="-6.985" y2="-11.7475" width="0.4064" layer="16"/>
-<wire x1="-6.985" y1="-11.7475" x2="-14.2875" y2="-11.7475" width="0.4064" layer="16"/>
-<wire x1="-14.2875" y1="-11.7475" x2="-15.24" y2="-11.43" width="0.4064" layer="16"/>
-<wire x1="-15.24" y1="-11.43" x2="-16.611578125" y2="-11.43" width="0.4064" layer="16"/>
-<wire x1="-16.611578125" y1="-11.43" x2="-16.612878125" y2="-11.4287" width="0.4064" layer="16"/>
 </signal>
 <signal name="VCC">
@@
 <wire x1="-17.1437" y1="-47.6237" x2="-14.605" y2="-45.085" width="0.4064" layer="16"/>
 <wire x1="-14.605" y1="-45.085" x2="-12.7" y2="-45.085" width="0.4064" layer="16"/>
-<wire x1="-13.971278125" y1="-39.4812" x2="-14.605" y2="-45.085" width="0" layer="19" extent="16-16"/>
+<wire x1="-13.971278125" y1="-39.4812" x2="-11.746221875" y2="-44.4513" width="0" layer="19" extent="16-16"/>
 </signal>
 <signal name="T3">
@@
 <wire x1="-22.86" y1="-50.8" x2="-23.4963" y2="-50.1637" width="0.4064" layer="16"/>
 <wire x1="-25.401278125" y1="-50.1637" x2="-23.4963" y2="-50.1637" width="0.4064" layer="16"/>
-<wire x1="-14.606278125" y1="-30.9087" x2="-13.97" y2="-47.625" width="0" layer="19" extent="16-16"/>
+<wire x1="-14.606278125" y1="-30.9087" x2="-11.746221875" y2="-46.9913" width="0" layer="19" extent="16-16"/>
 </signal>
 <signal name="T2">
@@
 <contactref element="DD3" pad="5"/>
 <wire x1="3.173721875" y1="-43.1787" x2="1.903721875" y2="-41.9087" width="0.4064" layer="16"/>
-<wire x1="1.903721875" y1="-41.9087" x2="1.903721875" y2="-39.3687" width="0.4064" layer="16"/>
+<wire x1="1.903721875" y1="-41.9087" x2="1.903721875" y2="-39.3687" width="0.3048" layer="16"/>
 <wire x1="1.903721875" y1="-39.3687" x2="3.173721875" y2="-38.0987" width="0.4064" layer="16"/>
 <wire x1="3.173721875" y1="-38.0987" x2="4.443721875" y2="-38.0987" width="0.4064" layer="16"/>
@@
 <contactref element="DD2" pad="1"/>
 <wire x1="5.713721875" y1="-43.1787" x2="6.983721875" y2="-41.9087" width="0.4064" layer="16"/>
-<wire x1="6.983721875" y1="-41.9087" x2="6.983721875" y2="-38.7337" width="0.4064" layer="16"/>
+<wire x1="6.983721875" y1="-41.9087" x2="6.983721875" y2="-38.7337" width="0.3048" layer="16"/>
 <wire x1="6.983721875" y1="-38.7337" x2="8.888721875" y2="-36.8287" width="0.4064" layer="16"/>
 <wire x1="8.888721875" y1="-36.8287" x2="12.063721875" y2="-36.8287" width="0.4064" layer="16"/>
@@
 <wire x1="3.173721875" y1="-40.6387" x2="3.173721875" y2="-40.0037" width="0.4064" layer="16"/>
 <wire x1="3.173721875" y1="-40.0037" x2="4.443721875" y2="-41.2737" width="0.4064" layer="16"/>
-<wire x1="4.443721875" y1="-41.2737" x2="4.443721875" y2="-45.0837" width="0.4064" layer="16"/>
+<wire x1="4.443721875" y1="-41.2737" x2="4.443721875" y2="-45.0837" width="0.3048" layer="16"/>
 <wire x1="4.443721875" y1="-45.0837" x2="5.713721875" y2="-45.7187" width="0.4064" layer="16"/>
 <wire x1="5.713721875" y1="-45.7187" x2="12.698721875" y2="-45.7187" width="0.4064" layer="16"/>
@@
 <wire x1="18.5437" y1="22.541221875" x2="18.376278125" y2="25.4462" width="0" layer="19" extent="16-16"/>
 <wire x1="22.5438" y1="23.683778125" x2="18.5437" y2="22.541221875" width="0" layer="19" extent="16-16"/>
-<wire x1="-6.18" y1="3.49" x2="18.5437" y2="22.541221875" width="0" layer="19" extent="16-16"/>
-<wire x1="-8.233778125" y1="-8.9912" x2="-6.18" y2="3.49" width="0" layer="19" extent="16-16"/>
+<wire x1="-5.8625" y1="3.49" x2="18.5437" y2="22.541221875" width="0" layer="19" extent="16-16"/>
+<wire x1="-8.233778125" y1="-8.9912" x2="-5.8625" y2="3.49" width="0" layer="19" extent="16-16"/>
 </signal>
 <signal name="SD">
@@
 <contactref element="DD4" pad="9"/>
 <wire x1="-3.191278125" y1="-2.54" x2="-3.191278125" y2="-0.2428" width="0.4064" layer="16"/>
-<wire x1="-3.98" y1="2.54" x2="-3.191278125" y2="2.54" width="0.4064" layer="16"/>
+<wire x1="-3.6625" y1="2.54" x2="-3.191278125" y2="2.54" width="0.4064" layer="16"/>
 <wire x1="-3.191278125" y1="2.54" x2="-3.191278125" y2="-0.2428" width="0.4064" layer="16"/>
+<contactref element="DD6" pad="9"/>
+<contactref element="U$58" pad="P$1"/>
+<wire x1="-4.7625" y1="-0.3175" x2="-22.759678125" y2="-11.4287" width="0" layer="19" extent="16-16"/>
+<wire x1="-4.7625" y1="-0.3175" x2="-3.191278125" y2="-0.3175" width="0.4064" layer="16"/>
+<wire x1="-3.191278125" y1="-0.3175" x2="-3.191278125" y2="-0.2428" width="0.4064" layer="16"/>
 </signal>
 <signal name="N$28">
